File: Powerboard/3.sch (KiCad schematic (older format))
At the start: 27 parts

Commit message: Updates changes 29/01/2022
Parts:
- C?: value C_Small -> 0.47μF
Changed lines of the file:
@@
 P 2750 5900
 F 0 "C?" H 2842 5946 50  0000 L CNN
-F 1 "C_Small" H 2842 5855 50  0000 L CNN
+F 1 "0.47μF" H 2842 5855 50  0000 L CNN
 F 2 "" H 2750 5900 50  0001 C CNN
 F 3 "~" H 2750 5900 50  0001 C CNN

Commit message: 01022022
Parts:
- removed C?: C_Small, symbol Device:C_Small
- removed Q? (x2): IRF7403, Package_SO:SOIC-8_3.9x4.9mm_P1.27mm, symbol Transistor_FET:IRF7403
- removed R?: R_Small, symbol Device:R_Small
- removed U?: LTC4370CMSTRPBF, MSOP-16_MS, symbol iclr:LTC4370CMSTRPBF
- added C?: 0.1µF, symbol Device:CP_Small
- added U?: LTC4412xS6, Package_TO_SOT_SMD:TSOT-23-6, symbol Power_Management:LTC4412xS6
Connections:
- wire segments 111 -> 93
Changed lines of the file:
@@
 $EndDescr
-$Comp
-L iclr:LTC4370CMSTRPBF U?
-U 1 1 61F114F7
-P 9300 2350
-AR Path="/61F114F7" Ref="U?"  Part="1"
-AR Path="/61F04C1A/61F114F7" Ref="U?"  Part="1"
-F 0 "U?" H 10700 2715 50  0000 C CNN
-F 1 "LTC4370CMSTRPBF" H 10700 2624 50  0000 C CNN
-F 2 "MSOP-16_MS" H 9300 2350 50  0001 L BNN
-F 3 "" H 9300 2350 50  0001 L BNN
-F 4 "ltc4370cms#trpbf" H 9300 2350 50  0001 L BNN "MANUFACTURER_PART_NUMBER"
-F 5 "Linear Technology" H 9300 2350 50  0001 L BNN "VENDOR"
-	1    9300 2350
-	0    1    1    0
-$EndComp
-$Comp
-L Transistor_FET:IRF7403 Q?
-U 1 1 61F1BB7A
-P 6900 5700
-F 0 "Q?" H 7105 5746 50  0000 L CNN
-F 1 "IRF7403" H 7105 5655 50  0000 L CNN
-F 2 "Package_SO:SOIC-8_3.9x4.9mm_P1.27mm" H 7100 5600 50  0001 L CNN
-F 3 "https://www.infineon.com/dgdl/irf7403pbf.pdf?fileId=5546d462533600a4015355fa23541b9c" H 6900 5700 50  0001 L CNN
-	1    6900 5700
-	0    1    1    0
-$EndComp
 $Comp
 L iclr:LM2679T-3.3 U?
@@
 U 1 1 61F105C2
 P 5100 6250
-F 0 "R?" H 5159 6296 50  0000 L CNN
-F 1 "R_Small" H 5159 6205 50  0000 L CNN
+F 0 "R?" H 4950 6300 50  0000 L CNN
+F 1 "R_Small" H 4900 6200 50  0000 L CNN
 F 2 "" H 5100 6250 50  0001 C CNN
 F 3 "~" H 5100 6250 50  0001 C CNN
@@
 U 1 1 61F1681B
 P 6300 6150
-F 0 "C?" V 6304 6253 50  0000 L CNN
-F 1 "C0603C103J5REC7411" V 6395 6253 50  0000 L CNN
+F 0 "C?" V 6250 5950 50  0000 L CNN
+F 1 "C0603C103J5REC7411" V 6550 5850 50  0000 L CNN
 F 2 "CAPC1608X87N" H 6300 6150 50  0001 L BNN
 F 3 "" H 6300 6150 50  0001 L BNN
@@
 Wire Wire Line
 	6550 5800 6700 5800
-$Comp
-L Transistor_FET:IRF7403 Q?
-U 1 1 61F3DFEB
-P 6850 900
-F 0 "Q?" H 7055 946 50  0000 L CNN
-F 1 "IRF7403" H 7055 855 50  0000 L CNN
-F 2 "Package_SO:SOIC-8_3.9x4.9mm_P1.27mm" H 7050 800 50  0001 L CNN
-F 3 "https://www.infineon.com/dgdl/irf7403pbf.pdf?fileId=5546d462533600a4015355fa23541b9c" H 6850 900 50  0001 L CNN
-	1    6850 900
-	0    1    1    0
-$EndComp
 $Comp
 L iclr:LM2679T-3.3 U?
@@
 U 1 1 61F3E071
 P 5050 1450
-F 0 "R?" H 5109 1496 50  0000 L CNN
-F 1 "R_Small" H 5109 1405 50  0000 L CNN
+F 0 "R?" H 4950 1500 50  0000 L CNN
+F 1 "R_Small" H 4850 1400 50  0000 L CNN
 F 2 "" H 5050 1450 50  0001 C CNN
 F 3 "~" H 5050 1450 50  0001 C CNN
@@
 U 1 1 61F3E08A
 P 6250 1350
-F 0 "C?" V 6254 1453 50  0000 L CNN
-F 1 "C0603C103J5REC7411" V 6345 1453 50  0000 L CNN
+F 0 "C?" V 6250 1150 50  0000 L CNN
+F 1 "C0603C103J5REC7411" V 6450 1000 50  0000 L CNN
 F 2 "CAPC1608X87N" H 6250 1350 50  0001 L BNN
 F 3 "" H 6250 1350 50  0001 L BNN
@@
 Wire Wire Line
 	6500 1250 6500 1000
-Connection ~ 6500 1000
 Wire Wire Line
 	1000 5800 1450 5800
@@
 Text HLabel 850  3750 0    50   Input ~ 0
 Vin
-$Comp
-L Device:R_Small R?
-U 1 1 61F45E94
-P 9200 2050
-F 0 "R?" H 9259 2096 50  0000 L CNN
-F 1 "R_Small" H 9259 2005 50  0000 L CNN
-F 2 "" H 9200 2050 50  0001 C CNN
-F 3 "~" H 9200 2050 50  0001 C CNN
-	1    9200 2050
-	1    0    0    -1
-$EndComp
-Wire Wire Line
-	9200 2350 9200 2150
-Wire Wire Line
-	9300 2350 9300 1950
-Wire Wire Line
-	9300 1950 9200 1950
-$Comp
-L power:GND #PWR?
-U 1 1 61F4AEBC
-P 9200 1800
-F 0 "#PWR?" H 9200 1550 50  0001 C CNN
-F 1 "GND" H 9205 1627 50  0000 C CNN
-F 2 "" H 9200 1800 50  0001 C CNN
-F 3 "" H 9200 1800 50  0001 C CNN
-	1    9200 1800
-	-1   0    0    1
-$EndComp
-Wire Wire Line
-	9200 1800 9200 1950
-Connection ~ 9200 1950
-$Comp
-L Device:C_Small C?
-U 1 1 61F4D8F5
-P 9100 5350
-F 0 "C?" H 9192 5396 50  0000 L CNN
-F 1 "C_Small" H 9192 5305 50  0000 L CNN
-F 2 "" H 9100 5350 50  0001 C CNN
-F 3 "~" H 9100 5350 50  0001 C CNN
-	1    9100 5350
-	1    0    0    -1
-$EndComp
-Wire Wire Line
-	9100 5150 9100 5250
-Wire Wire Line
-	9200 5150 9200 5450
-Wire Wire Line
-	9200 5450 9100 5450
-$Comp
-L power:GND #PWR?
-U 1 1 61F5293F
-P 9100 5450
-F 0 "#PWR?" H 9100 5200 50  0001 C CNN
-F 1 "GND" H 9105 5277 50  0000 C CNN
-F 2 "" H 9100 5450 50  0001 C CNN
-F 3 "" H 9100 5450 50  0001 C CNN
-	1    9100 5450
-	1    0    0    -1
-$EndComp
-$Comp
-L power:GND #PWR?
-U 1 1 61F55478
-P 9300 5250
-F 0 "#PWR?" H 9300 5000 50  0001 C CNN
-F 1 "GND" H 9305 5077 50  0000 C CNN
-F 2 "" H 9300 5250 50  0001 C CNN
-F 3 "" H 9300 5250 50  0001 C CNN
-	1    9300 5250
-	1    0    0    -1
-$EndComp
-Wire Wire Line
-	9300 5150 9300 5250
-Wire Wire Line
-	8900 5150 8900 5500
-Wire Wire Line
-	8900 5500 6900 5500
 Text HLabel 10500 3700 2    50   Input ~ 0
 Vout
 Wire Wire Line
 	7100 5800 10150 5800
-Connection ~ 9100 5450
 Wire Wire Line
 	1000 1000 1000 3750
 Connection ~ 1000 3750
 Wire Wire Line
-	6850 700  8900 700
-Wire Wire Line
-	8900 700  8900 2350
-Wire Wire Line
-	7050 1000 10150 1000
-Wire Wire Line
 	10150 1000 10150 3700
-Wire Wire Line
-	6500 1000 6600 1000
-Wire Wire Line
-	9000 2350 9000 1200
-Wire Wire Line
-	9000 1200 6600 1200
-Wire Wire Line
-	6600 1200 6600 1000
-Connection ~ 6600 1000
-Wire Wire Line
-	6600 1000 6650 1000
-Wire Wire Line
-	6700 5800 6700 5950
-Wire Wire Line
-	6700 5950 9000 5950
-Wire Wire Line
-	9000 5950 9000 5150
-Connection ~ 6700 5800
 Wire Wire Line
 	10500 3700 10150 3700
@@
 Wire Wire Line
 	10150 3700 10150 5800
+Connection ~ 6500 1000
+$Comp
+L Power_Management:LTC4412xS6 U?
+U 1 1 620B10E4
+P 7900 1850
+F 0 "U?" H 7550 1300 50  0000 C CNN
+F 1 "LTC4412xS6" H 7550 1400 50  0000 C CNN
+F 2 "Package_TO_SOT_SMD:TSOT-23-6" H 8550 1500 50  0001 C CNN
+F 3 "https://www.analog.com/media/en/technical-documentation/data-sheets/4412fb.pdf" H 10000 1650 50  0001 C CNN
+	1    7900 1850
+	1    0    0    -1
+$EndComp
+Wire Wire Line
+	7500 1000 7500 1750
+Wire Wire Line
+	6500 1000 7500 1000
+$Comp
+L power:GND #PWR?
+U 1 1 620BB43D
+P 7900 2250
+F 0 "#PWR?" H 7900 2000 50  0001 C CNN
+F 1 "GND" V 7905 2122 50  0000 R CNN
+F 2 "" H 7900 2250 50  0001 C CNN
+F 3 "" H 7900 2250 50  0001 C CNN
+	1    7900 2250
+	1    0    0    -1
+$EndComp
+$Comp
+L Device:CP_Small C?
+U 1 1 620BC376
+P 7350 1750
+F 0 "C?" V 7125 1750 50  0000 C CNN
+F 1 "0.1µF" V 7216 1750 50  0000 C CNN
+F 2 "" H 7350 1750 50  0001 C CNN
+F 3 "~" H 7350 1750 50  0001 C CNN
+	1    7350 1750
+	0    1    1    0
+$EndComp
+$Comp
+L power:GND #PWR?
+U 1 1 620B8A1A
+P 7250 1750
+F 0 "#PWR?" H 7250 1500 50  0001 C CNN
+F 1 "GND" V 7255 1622 50  0000 R CNN
+F 2 "" H 7250 1750 50  0001 C CNN
+F 3 "" H 7250 1750 50  0001 C CNN
+	1    7250 1750
+	0    1    1    0
+$EndComp
+Wire Wire Line
+	7450 1750 7500 1750
+Connection ~ 7500 1750
 $EndSCHEMATC
