File: Powerboard/3.sch (KiCad schematic (older format))
At the start: 25 parts

Commit message: 08/02/2022 update
Parts:
- added Q? (x2): CSD25485F5T, CSD13385F5, symbol iclr:CSD25485F5T
Connections:
- wire segments 92 -> 103
Other:
- moved on the sheet: U?
Changed lines of the file:
@@
 Wire Wire Line
 	6550 6050 6550 5800
-Connection ~ 6550 5800
 $Comp
 L iclr:LM2679T-3.3 U?
@@
 Connection ~ 1000 3750
 Wire Wire Line
-	10150 1000 10150 3700
-Wire Wire Line
 	10500 3700 10150 3700
 Connection ~ 10150 3700
@@
 L Power_Management:LTC4412xS6 U?
 U 1 1 61FEA01F
-P 7650 5900
-F 0 "U?" H 7300 5350 50  0000 C CNN
-F 1 "LTC4412xS6" H 7300 5450 50  0000 C CNN
-F 2 "Package_TO_SOT_SMD:TSOT-23-6" H 8300 5550 50  0001 C CNN
-F 3 "https://www.analog.com/media/en/technical-documentation/data-sheets/4412fb.pdf" H 9750 5700 50  0001 C CNN
-	1    7650 5900
-	1    0    0    -1
-$EndComp
-Wire Wire Line
-	6550 5800 7250 5800
+P 7850 5250
+F 0 "U?" H 7500 4700 50  0000 C CNN
+F 1 "LTC4412xS6" H 7500 4800 50  0000 C CNN
+F 2 "Package_TO_SOT_SMD:TSOT-23-6" H 8500 4900 50  0001 C CNN
+F 3 "https://www.analog.com/media/en/technical-documentation/data-sheets/4412fb.pdf" H 9950 5050 50  0001 C CNN
+	1    7850 5250
+	1    0    0    -1
+$EndComp
+Wire Wire Line
+	6750 5150 7450 5150
 $Comp
 L power:GND #PWR?
@@
 	1    0    0    -1
 $EndComp
+$Comp
+L iclr:CSD25485F5T Q?
+U 1 1 6202F74F
+P 8450 1050
+F 0 "Q?" V 8925 1150 50  0000 C CNN
+F 1 "CSD25485F5T" V 9016 1150 50  0000 C CNN
+F 2 "CSD13385F5" H 8900 1000 50  0001 L CNN
+F 3 "http://www.ti.com/lit/gpn/CSD25485F5" H 8900 900 50  0001 L CNN
+F 4 "-20V, P ch NexFET MOSFET, single LGA 0.8x1.5, 42mOhm" H 8900 800 50  0001 L CNN "Description"
+F 5 "0" H 8900 700 50  0001 L CNN "Height"
+F 6 "Texas Instruments" H 8900 600 50  0001 L CNN "Manufacturer_Name"
+F 7 "CSD25485F5T" H 8900 500 50  0001 L CNN "Manufacturer_Part_Number"
+F 8 "595-CSD25485F5T" H 8900 400 50  0001 L CNN "Mouser Part Number"
+F 9 "https://www.mouser.co.uk/ProductDetail/Texas-Instruments/CSD25485F5T?qs=Bho%2FbeBaDExWIlvMtFx97A%3D%3D" H 8900 300 50  0001 L CNN "Mouser Price/Stock"
+F 10 "CSD25485F5T" H 8900 200 50  0001 L CNN "Arrow Part Number"
+F 11 "https://www.arrow.com/en/products/csd25485f5t/texas-instruments" H 8900 100 50  0001 L CNN "Arrow Price/Stock"
+	1    8450 1050
+	0    1    1    0
+$EndComp
+Wire Wire Line
+	7500 1000 8250 1000
+Wire Wire Line
+	8250 1000 8250 1350
+Connection ~ 7500 1000
+Wire Wire Line
+	8450 1050 7900 1050
+Wire Wire Line
+	7900 1050 7900 1450
+Wire Wire Line
+	8850 1350 10150 1350
+Wire Wire Line
+	10150 1350 10150 3700
+$Comp
+L power:GND #PWR?
+U 1 1 6203E5CB
+P 7500 1950
+F 0 "#PWR?" H 7500 1700 50  0001 C CNN
+F 1 "GND" V 7505 1822 50  0000 R CNN
+F 2 "" H 7500 1950 50  0001 C CNN
+F 3 "" H 7500 1950 50  0001 C CNN
+	1    7500 1950
+	0    1    1    0
+$EndComp
+$Comp
+L power:GND #PWR?
+U 1 1 6203EB10
+P 7450 5350
+F 0 "#PWR?" H 7450 5100 50  0001 C CNN
+F 1 "GND" V 7455 5222 50  0000 R CNN
+F 2 "" H 7450 5350 50  0001 C CNN
+F 3 "" H 7450 5350 50  0001 C CNN
+	1    7450 5350
+	0    1    1    0
+$EndComp
+$Comp
+L iclr:CSD25485F5T Q?
+U 1 1 6203F31D
+P 8650 5500
+F 0 "Q?" V 9125 5600 50  0000 C CNN
+F 1 "CSD25485F5T" V 9216 5600 50  0000 C CNN
+F 2 "CSD13385F5" H 9100 5450 50  0001 L CNN
+F 3 "http://www.ti.com/lit/gpn/CSD25485F5" H 9100 5350 50  0001 L CNN
+F 4 "-20V, P ch NexFET MOSFET, single LGA 0.8x1.5, 42mOhm" H 9100 5250 50  0001 L CNN "Description"
+F 5 "0" H 9100 5150 50  0001 L CNN "Height"
+F 6 "Texas Instruments" H 9100 5050 50  0001 L CNN "Manufacturer_Name"
+F 7 "CSD25485F5T" H 9100 4950 50  0001 L CNN "Manufacturer_Part_Number"
+F 8 "595-CSD25485F5T" H 9100 4850 50  0001 L CNN "Mouser Part Number"
+F 9 "https://www.mouser.co.uk/ProductDetail/Texas-Instruments/CSD25485F5T?qs=Bho%2FbeBaDExWIlvMtFx97A%3D%3D" H 9100 4750 50  0001 L CNN "Mouser Price/Stock"
+F 10 "CSD25485F5T" H 9100 4650 50  0001 L CNN "Arrow Part Number"
+F 11 "https://www.arrow.com/en/products/csd25485f5t/texas-instruments" H 9100 4550 50  0001 L CNN "Arrow Price/Stock"
+	1    8650 5500
+	0    1    1    0
+$EndComp
+Wire Wire Line
+	6750 5150 6750 5800
+Wire Wire Line
+	6750 5800 6550 5800
+Connection ~ 6550 5800
+Wire Wire Line
+	6750 5800 8450 5800
+Connection ~ 6750 5800
+Wire Wire Line
+	7850 4850 8650 4850
+Wire Wire Line
+	8650 4850 8650 5500
+Wire Wire Line
+	9050 5800 10150 5800
+$Comp
+L power:GND #PWR?
+U 1 1 62050F8C
+P 7850 5650
+F 0 "#PWR?" H 7850 5400 50  0001 C CNN
+F 1 "GND" H 7855 5477 50  0000 C CNN
+F 2 "" H 7850 5650 50  0001 C CNN
+F 3 "" H 7850 5650 50  0001 C CNN
+	1    7850 5650
+	1    0    0    -1
+$EndComp

Commit message: 08/02/2022
3.3v regulators complete
Parts:
- added C?: 0.1µF, symbol Device:CP_Small
Connections:
- net labels added: STAT1, STAT2
Changed lines of the file:
@@
 U 1 1 61F1681B
 P 6300 6150
+AR Path="/61F1681B" Ref="C?"  Part="1"
+AR Path="/61F04C1A/61F1681B" Ref="C?"  Part="1"
 F 0 "C?" V 6250 5950 50  0000 L CNN
 F 1 "C0603C103J5REC7411" V 6550 5850 50  0000 L CNN
@@
 U 1 1 61F17164
 P 6550 6150
+AR Path="/61F17164" Ref="C?"  Part="1"
+AR Path="/61F04C1A/61F17164" Ref="C?"  Part="1"
 F 0 "C?" V 6554 6253 50  0000 L CNN
 F 1 "C0603C103J5REC7411" V 6645 6253 50  0000 L CNN
@@
 U 1 1 61F3E08A
 P 6250 1350
+AR Path="/61F3E08A" Ref="C?"  Part="1"
+AR Path="/61F04C1A/61F3E08A" Ref="C?"  Part="1"
 F 0 "C?" V 6250 1150 50  0000 L CNN
 F 1 "C0603C103J5REC7411" V 6450 1000 50  0000 L CNN
@@
 U 1 1 61F3E090
 P 6500 1350
+AR Path="/61F3E090" Ref="C?"  Part="1"
+AR Path="/61F04C1A/61F3E090" Ref="C?"  Part="1"
 F 0 "C?" V 6504 1453 50  0000 L CNN
 F 1 "C0603C103J5REC7411" V 6595 1453 50  0000 L CNN
@@
 	1    0    0    -1
 $EndComp
+$Comp
+L power:GND #PWR?
+U 1 1 6202F9B8
+P 8300 1750
+F 0 "#PWR?" H 8300 1500 50  0001 C CNN
+F 1 "GND" V 8305 1622 50  0000 R CNN
+F 2 "" H 8300 1750 50  0001 C CNN
+F 3 "" H 8300 1750 50  0001 C CNN
+	1    8300 1750
+	0    -1   -1   0
+$EndComp
+Text HLabel 8300 1950 2    50   Input ~ 0
+STAT1
+$Comp
+L power:GND #PWR?
+U 1 1 620307B8
+P 8250 5150
+F 0 "#PWR?" H 8250 4900 50  0001 C CNN
+F 1 "GND" V 8255 5022 50  0000 R CNN
+F 2 "" H 8250 5150 50  0001 C CNN
+F 3 "" H 8250 5150 50  0001 C CNN
+	1    8250 5150
+	0    -1   -1   0
+$EndComp
+$Comp
+L Device:CP_Small C?
+U 1 1 62031A96
+P 6650 5150
+F 0 "C?" V 6425 5150 50  0000 C CNN
+F 1 "0.1µF" V 6516 5150 50  0000 C CNN
+F 2 "" H 6650 5150 50  0001 C CNN
+F 3 "~" H 6650 5150 50  0001 C CNN
+	1    6650 5150
+	0    1    1    0
+$EndComp
+Connection ~ 6750 5150
+$Comp
+L power:GND #PWR?
+U 1 1 62031F5A
+P 6550 5150
+F 0 "#PWR?" H 6550 4900 50  0001 C CNN
+F 1 "GND" V 6555 5022 50  0000 R CNN
+F 2 "" H 6550 5150 50  0001 C CNN
+F 3 "" H 6550 5150 50  0001 C CNN
+	1    6550 5150
+	0    1    1    0
+$EndComp
+Text HLabel 8250 5350 2    50   Input ~ 0
+STAT2
 $EndSCHEMATC

Commit message: reverse polarity protection
Connections:
- wire segments 103 -> 115
- no-connect marks 0 -> 4
Changed lines of the file:
@@
 U 1 1 620B10E4
 P 7900 1850
-F 0 "U?" H 7550 1300 50  0000 C CNN
-F 1 "LTC4412xS6" H 7550 1400 50  0000 C CNN
+F 0 "U?" H 8300 1350 50  0000 C CNN
+F 1 "LTC4412xS6" H 8250 1450 50  0000 C CNN
 F 2 "Package_TO_SOT_SMD:TSOT-23-6" H 8550 1500 50  0001 C CNN
 F 3 "https://www.analog.com/media/en/technical-documentation/data-sheets/4412fb.pdf" H 10000 1650 50  0001 C CNN
@@
 L power:GND #PWR?
 U 1 1 620BB43D
-P 7900 2250
-F 0 "#PWR?" H 7900 2000 50  0001 C CNN
-F 1 "GND" V 7905 2122 50  0000 R CNN
-F 2 "" H 7900 2250 50  0001 C CNN
-F 3 "" H 7900 2250 50  0001 C CNN
-	1    7900 2250
+P 7900 2350
+F 0 "#PWR?" H 7900 2100 50  0001 C CNN
+F 1 "GND" V 7905 2222 50  0000 R CNN
+F 2 "" H 7900 2350 50  0001 C CNN
+F 3 "" H 7900 2350 50  0001 C CNN
+	1    7900 2350
 	1    0    0    -1
 $EndComp
@@
 	7900 1050 7900 1450
 Wire Wire Line
-	8850 1350 10150 1350
+	8850 1350 9000 1350
 Wire Wire Line
 	10150 1350 10150 3700
 $Comp
 L power:GND #PWR?
-U 1 1 6203E5CB
-P 7500 1950
-F 0 "#PWR?" H 7500 1700 50  0001 C CNN
-F 1 "GND" V 7505 1822 50  0000 R CNN
-F 2 "" H 7500 1950 50  0001 C CNN
-F 3 "" H 7500 1950 50  0001 C CNN
-	1    7500 1950
-	0    1    1    0
-$EndComp
-$Comp
-L power:GND #PWR?
 U 1 1 6203EB10
-P 7450 5350
-F 0 "#PWR?" H 7450 5100 50  0001 C CNN
-F 1 "GND" V 7455 5222 50  0000 R CNN
-F 2 "" H 7450 5350 50  0001 C CNN
-F 3 "" H 7450 5350 50  0001 C CNN
-	1    7450 5350
+P 7300 5350
+F 0 "#PWR?" H 7300 5100 50  0001 C CNN
+F 1 "GND" V 7305 5222 50  0000 R CNN
+F 2 "" H 7300 5350 50  0001 C CNN
+F 3 "" H 7300 5350 50  0001 C CNN
+	1    7300 5350
 	0    1    1    0
 $EndComp
@@
 	8650 4850 8650 5500
 Wire Wire Line
-	9050 5800 10150 5800
-$Comp
-L power:GND #PWR?
-U 1 1 62050F8C
-P 7850 5650
-F 0 "#PWR?" H 7850 5400 50  0001 C CNN
-F 1 "GND" H 7855 5477 50  0000 C CNN
-F 2 "" H 7850 5650 50  0001 C CNN
-F 3 "" H 7850 5650 50  0001 C CNN
-	1    7850 5650
-	1    0    0    -1
-$EndComp
-$Comp
-L power:GND #PWR?
-U 1 1 6202F9B8
-P 8300 1750
-F 0 "#PWR?" H 8300 1500 50  0001 C CNN
-F 1 "GND" V 8305 1622 50  0000 R CNN
-F 2 "" H 8300 1750 50  0001 C CNN
-F 3 "" H 8300 1750 50  0001 C CNN
-	1    8300 1750
-	0    -1   -1   0
-$EndComp
+	9050 5800 9200 5800
 Text HLabel 8300 1950 2    50   Input ~ 0
 STAT1
-$Comp
-L power:GND #PWR?
-U 1 1 620307B8
-P 8250 5150
-F 0 "#PWR?" H 8250 4900 50  0001 C CNN
-F 1 "GND" V 8255 5022 50  0000 R CNN
-F 2 "" H 8250 5150 50  0001 C CNN
-F 3 "" H 8250 5150 50  0001 C CNN
-	1    8250 5150
-	0    -1   -1   0
-$EndComp
 $Comp
 L Device:CP_Small C?
@@
 Text HLabel 8250 5350 2    50   Input ~ 0
 STAT2
+Wire Wire Line
+	8300 1750 9000 1750
+Wire Wire Line
+	9000 1750 9000 1350
+Connection ~ 9000 1350
+Wire Wire Line
+	9000 1350 10150 1350
+Wire Wire Line
+	8250 5150 9200 5150
+Wire Wire Line
+	9200 5150 9200 5800
+Connection ~ 9200 5800
+Wire Wire Line
+	9200 5800 10150 5800
+Wire Wire Line
+	7850 5650 7300 5650
+Wire Wire Line
+	7300 5650 7300 5350
+Wire Wire Line
+	7450 5350 7300 5350
+Connection ~ 7300 5350
+Wire Wire Line
+	7500 2350 7900 2350
+Wire Wire Line
+	7500 1950 7500 2350
+Wire Wire Line
+	7900 2250 7900 2350
+Connection ~ 7900 2350
+NoConn ~ 4950 1200
+NoConn ~ 3150 1100
+NoConn ~ 3200 5900
+NoConn ~ 5000 6000
 $EndSCHEMATC

Commit message: 13/02/2022
reverse polarity protection added, some test points, general clear up
Parts:
- C? (x8): symbol iclr:EEUFM1H471 -> power_new_25012022-rescue:EEUFM1H471-iclr
- C? (x4): symbol iclr:C0603C103J5REC7411 -> power_new_25012022-rescue:C0603C103J5REC7411-iclr
- D? (x2): symbol iclr:MBRD835LT4G -> power_new_25012022-rescue:MBRD835LT4G-iclr
- L? (x2): symbol iclr:P0846SNL -> power_new_25012022-rescue:P0846SNL-iclr
- Q? (x2): symbol iclr:CSD25485F5T -> power_new_25012022-rescue:CSD25485F5T-iclr
- U? (x2): symbol iclr:LM2679T-3.3 -> power_new_25012022-rescue:LM2679T-3.3-iclr
Changed lines of the file:
@@
 $EndDescr
 $Comp
-L iclr:LM2679T-3.3 U?
+L power_new_25012022-rescue:LM2679T-3.3-iclr U?
 U 1 1 61F11502
 P 4100 5800
@@
 Connection ~ 1450 5800
 $Comp
-L iclr:EEUFM1H471 C?
+L power_new_25012022-rescue:EEUFM1H471-iclr C?
 U 1 1 61F06827
 P 1450 6050
@@
 $EndComp
 $Comp
-L iclr:EEUFM1H471 C?
+L power_new_25012022-rescue:EEUFM1H471-iclr C?
 U 1 1 61F07F24
 P 1800 6050
@@
 	1800 5800 1450 5800
 $Comp
-L iclr:EEUFM1H471 C?
+L power_new_25012022-rescue:EEUFM1H471-iclr C?
 U 1 1 61F0A525
 P 2150 6050
@@
 $EndComp
 $Comp
-L iclr:EEUFM1H471 C?
+L power_new_25012022-rescue:EEUFM1H471-iclr C?
 U 1 1 61F0A533
 P 2500 6050
@@
 	3100 6450 3100 6550
 $Comp
-L iclr:P0846SNL L?
+L power_new_25012022-rescue:P0846SNL-iclr L?
 U 1 1 61F0F3B2
 P 5350 5800
@@
 	5350 5800 5300 5800
 $Comp
-L iclr:MBRD835LT4G D?
+L power_new_25012022-rescue:MBRD835LT4G-iclr D?
 U 1 1 61F1381F
 P 5300 6250
@@
 	5300 5800 5000 5800
 $Comp
-L iclr:C0603C103J5REC7411 C?
+L power_new_25012022-rescue:C0603C103J5REC7411-iclr C?
 U 1 1 61F1681B
 P 6300 6150
@@
 $EndComp
 $Comp
-L iclr:C0603C103J5REC7411 C?
+L power_new_25012022-rescue:C0603C103J5REC7411-iclr C?
 U 1 1 61F17164
 P 6550 6150
@@
 	6550 6050 6550 5800
 $Comp
-L iclr:LM2679T-3.3 U?
+L power_new_25012022-rescue:LM2679T-3.3-iclr U?
 U 1 1 61F3DFF6
 P 4050 1000
@@
 Connection ~ 1400 1000
 $Comp
-L iclr:EEUFM1H471 C?
+L power_new_25012022-rescue:EEUFM1H471-iclr C?
 U 1 1 61F3E007
 P 1400 1250
@@
 $EndComp
 $Comp
-L iclr:EEUFM1H471 C?
+L power_new_25012022-rescue:EEUFM1H471-iclr C?
 U 1 1 61F3E015
 P 1750 1250
@@
 	1750 1000 1400 1000
 $Comp
-L iclr:EEUFM1H471 C?
+L power_new_25012022-rescue:EEUFM1H471-iclr C?
 U 1 1 61F3E026
 P 2100 1250
@@
 $EndComp
 $Comp
-L iclr:EEUFM1H471 C?
+L power_new_25012022-rescue:EEUFM1H471-iclr C?
 U 1 1 61F3E034
 P 2450 1250
@@
 	3050 1650 3050 1750
 $Comp
-L iclr:P0846SNL L?
+L power_new_25012022-rescue:P0846SNL-iclr L?
 U 1 1 61F3E06B
 P 5300 1000
@@
 	5300 1000 5250 1000
 $Comp
-L iclr:MBRD835LT4G D?
+L power_new_25012022-rescue:MBRD835LT4G-iclr D?
 U 1 1 61F3E07D
 P 5250 1450
@@
 	5250 1000 4950 1000
 $Comp
-L iclr:C0603C103J5REC7411 C?
+L power_new_25012022-rescue:C0603C103J5REC7411-iclr C?
 U 1 1 61F3E08A
 P 6250 1350
@@
 $EndComp
 $Comp
-L iclr:C0603C103J5REC7411 C?
+L power_new_25012022-rescue:C0603C103J5REC7411-iclr C?
 U 1 1 61F3E090
 P 6500 1350
@@
 	6750 5150 7450 5150
 $Comp
-L power:GND #PWR?
-U 1 1 61FED494
-P 7650 6300
-F 0 "#PWR?" H 7650 6050 50  0001 C CNN
-F 1 "GND" H 7655 6127 50  0000 C CNN
-F 2 "" H 7650 6300 50  0001 C CNN
-F 3 "" H 7650 6300 50  0001 C CNN
-	1    7650 6300
-	1    0    0    -1
-$EndComp
-$Comp
-L iclr:CSD25485F5T Q?
+L power_new_25012022-rescue:CSD25485F5T-iclr Q?
 U 1 1 6202F74F
 P 8450 1050
@@
 $EndComp
 $Comp
-L iclr:CSD25485F5T Q?
+L power_new_25012022-rescue:CSD25485F5T-iclr Q?
 U 1 1 6203F31D
 P 8650 5500

Commit message: 13/02/2022
Parts:
- added TP? (x4): TestPoint, symbol Connector:TestPoint
Connections:
- net Vin: now also TP?.1, TP?.1
- net Vout: now also TP?.1, TP?.1
Changed lines of the file:
@@
 Connection ~ 2750 5800
 Wire Wire Line
-	2750 5800 3200 5800
+	2750 5800 3100 5800
 Wire Wire Line
 	1800 5800 2150 5800
@@
 Connection ~ 2700 1000
 Wire Wire Line
-	2700 1000 3150 1000
+	2700 1000 2950 1000
 Wire Wire Line
 	1750 1000 2100 1000
@@
 	1000 5800 1450 5800
 Wire Wire Line
-	1000 3750 850  3750
-Wire Wire Line
 	1000 3750 1000 5800
-Text HLabel 850  3750 0    50   Input ~ 0
+Text HLabel 700  3750 0    50   Input ~ 0
 Vin
 Text HLabel 10500 3700 2    50   Input ~ 0
@@
 Connection ~ 9000 1350
 Wire Wire Line
-	9000 1350 10150 1350
+	9000 1350 9250 1350
 Wire Wire Line
 	8250 5150 9200 5150
@@
 Connection ~ 9200 5800
 Wire Wire Line
-	9200 5800 10150 5800
+	9200 5800 9450 5800
 Wire Wire Line
 	7850 5650 7300 5650
@@
 NoConn ~ 3200 5900
 NoConn ~ 5000 6000
+$Comp
+L Connector:TestPoint TP?
+U 1 1 620D20B1
+P 9250 1350
+F 0 "TP?" H 9308 1468 50  0000 L CNN
+F 1 "TestPoint" H 9308 1377 50  0000 L CNN
+F 2 "" H 9450 1350 50  0001 C CNN
+F 3 "~" H 9450 1350 50  0001 C CNN
+	1    9250 1350
+	1    0    0    -1
+$EndComp
+Connection ~ 9250 1350
+Wire Wire Line
+	9250 1350 10150 1350
+$Comp
+L Connector:TestPoint TP?
+U 1 1 620D24CD
+P 9450 5800
+F 0 "TP?" H 9392 5826 50  0000 R CNN
+F 1 "TestPoint" H 9392 5917 50  0000 R CNN
+F 2 "" H 9650 5800 50  0001 C CNN
+F 3 "~" H 9650 5800 50  0001 C CNN
+	1    9450 5800
+	-1   0    0    1
+$EndComp
+Connection ~ 9450 5800
+Wire Wire Line
+	9450 5800 10150 5800
+Wire Wire Line
+	700  3750 1000 3750
+$Comp
+L Connector:TestPoint TP?
+U 1 1 620D653C
+P 2950 1000
+F 0 "TP?" H 3008 1118 50  0000 L CNN
+F 1 "TestPoint" H 3008 1027 50  0000 L CNN
+F 2 "" H 3150 1000 50  0001 C CNN
+F 3 "~" H 3150 1000 50  0001 C CNN
+	1    2950 1000
+	1    0    0    -1
+$EndComp
+Connection ~ 2950 1000
+Wire Wire Line
+	2950 1000 3150 1000
+$Comp
+L Connector:TestPoint TP?
+U 1 1 620D69CA
+P 3100 5800
+F 0 "TP?" H 3158 5918 50  0000 L CNN
+F 1 "TestPoint" H 3158 5827 50  0000 L CNN
+F 2 "" H 3300 5800 50  0001 C CNN
+F 3 "~" H 3300 5800 50  0001 C CNN
+	1    3100 5800
+	1    0    0    -1
+$EndComp
+Connection ~ 3100 5800
+Wire Wire Line
+	3100 5800 3200 5800
 $EndSCHEMATC

Commit message: 19/02/2022
Parts:
- removed C? (x8): EEUFM1H471, CAPPRD500W60D1250H2000, symbol power_new_25012022-rescue:EEUFM1H471-iclr
- removed C? (x4): C0603C103J5REC7411, CAPC1608X87N, symbol power_new_25012022-rescue:C0603C103J5REC7411-iclr
- removed D? (x2): MBRD835LT4G, DPAK229P990X238-3N, symbol power_new_25012022-rescue:MBRD835LT4G-iclr
- removed L? (x2): P0846SNL, P0846SNL, symbol power_new_25012022-rescue:P0846SNL-iclr
- removed Q? (x2): CSD25485F5T, CSD13385F5, symbol power_new_25012022-rescue:CSD25485F5T-iclr
- removed U? (x2): LM2679T-3.3, TO127P457X1016X2052-7P, symbol power_new_25012022-rescue:LM2679T-3.3-iclr
- added C? (x4): C0603C103J5REC7411-iclr, CAPC1608X87N, symbol iclr:C0603C103J5REC7411-iclr
- added C? (x8): EEUFM1H471-iclr, CAPPRD500W60D1250H2000, symbol iclr:EEUFM1H471-iclr
- added D? (x2): MBRD835LT4G-iclr, DPAK229P990X238-3N, symbol iclr:MBRD835LT4G-iclr
- added L? (x2): P0846SNL-iclr, P0846SNL, symbol iclr:P0846SNL-iclr
- added Q? (x2): CSD25485F5T-iclr, CSD13385F5, symbol iclr:CSD25485F5T-iclr
- added U? (x2): LM2679T-3.3-iclr, TO127P457X1016X2052-7P, symbol iclr:LM2679T-3.3-iclr
Connections:
- net GND: now also C?.2, C?.2, C?.2, C?.2, C?.N, C?.N, C?.N, C?.N, C?.N, C?.N, C?.N, C?.N, D?.1, D?.1, D?.3, D?.3, U?.4 (GND), U?.4 (GND)
- net Vin: now also C?.P, C?.P, C?.P, C?.P, C?.P, C?.P, C?.P, C?.P, U?.2 (VIN), U?.2 (VIN)
- net Vout: now also Q?.3, Q?.3
- net at C?.1, U?.1 (VIN): now also C?.1, C?.1, L?.2, Q?.2, U?.6 (FB) (x2)
- net at R?.1: now also U?.5 (CURRENT_ADJ) (x2)
- net at U?.5 (GATE): now also Q?.1 (x2)
- new net: D?.4, L?.1, U?.1 (SW) (x2)
