File: Powerboard/_autosave-3.sch (KiCad schematic (older format))
At the start: 25 parts

Commit message: 05/02/2022
Parts:
- added C?: 0.1µF, symbol Device:CP_Small
- added Q? (x2): CSD25485F5T, CSD13385F5, symbol iclr:CSD25485F5T
- gave numbers to parts that had none: 1
Connections:
- net labels added: STAT1, STAT2
- wire segments 92 -> 102
Other:
- moved on the sheet: U?
Changed lines of the file:
@@
 Wire Wire Line
 	6550 6050 6550 5800
-Connection ~ 6550 5800
 $Comp
 L iclr:LM2679T-3.3 U?
@@
 Connection ~ 1400 1000
 $Comp
-L iclr:EEUFM1H471 C?
+L iclr:EEUFM1H471 CIN
 U 1 1 61F3E007
 P 1400 1250
-F 0 "C?" V 1400 950 50  0000 L CNN
-F 1 "EEUFM1H471" V 1700 950 50  0000 L CNN
+F 0 "CIN" V 1450 950 50  0000 L CNN
+F 1 "EEUFM1H471" V 1600 750 50  0000 L CNN
 F 2 "CAPPRD500W60D1250H2000" H 1400 1250 50  0001 L BNN
 F 3 "" H 1400 1250 50  0001 L BNN
@@
 $EndComp
 $Comp
-L iclr:EEUFM1H471 C?
+L iclr:EEUFM1H471 CIN
 U 1 1 61F3E015
 P 1750 1250
-F 0 "C?" V 1750 950 50  0000 L CNN
+F 0 "CIN" V 1950 1100 50  0000 L CNN
 F 1 "EEUFM1H471" V 2050 950 50  0000 L CNN
 F 2 "CAPPRD500W60D1250H2000" H 1750 1250 50  0001 L BNN
@@
 	1750 1000 1400 1000
 $Comp
-L iclr:EEUFM1H471 C?
+L iclr:EEUFM1H471 CIN
 U 1 1 61F3E026
 P 2100 1250
-F 0 "C?" V 2100 950 50  0000 L CNN
-F 1 "EEUFM1H471" V 2400 950 50  0000 L CNN
+F 0 "CIN" V 2200 1150 50  0000 L CNN
+F 1 "EEUFM1H471" V 2300 1100 50  0000 L CNN
 F 2 "CAPPRD500W60D1250H2000" H 2100 1250 50  0001 L BNN
 F 3 "" H 2100 1250 50  0001 L BNN
@@
 $EndComp
 $Comp
-L iclr:EEUFM1H471 C?
+L iclr:EEUFM1H471 CIN
 U 1 1 61F3E034
 P 2450 1250
-F 0 "C?" V 2450 950 50  0000 L CNN
-F 1 "EEUFM1H471" V 2750 950 50  0000 L CNN
+F 0 "CIN" V 2550 1450 50  0000 L CNN
+F 1 "EEUFM1H471" V 2650 1400 50  0000 L CNN
 F 2 "CAPPRD500W60D1250H2000" H 2450 1250 50  0001 L BNN
 F 3 "" H 2450 1250 50  0001 L BNN
@@
 Wire Wire Line
 	10500 3700 10150 3700
-Connection ~ 10150 3700
-Wire Wire Line
-	10150 3700 10150 5800
 Connection ~ 6500 1000
 $Comp
@@
 L Power_Management:LTC4412xS6 U?
 U 1 1 61FEA01F
-P 7650 5900
-F 0 "U?" H 7300 5350 50  0000 C CNN
-F 1 "LTC4412xS6" H 7300 5450 50  0000 C CNN
-F 2 "Package_TO_SOT_SMD:TSOT-23-6" H 8300 5550 50  0001 C CNN
-F 3 "https://www.analog.com/media/en/technical-documentation/data-sheets/4412fb.pdf" H 9750 5700 50  0001 C CNN
-	1    7650 5900
-	1    0    0    -1
-$EndComp
-Wire Wire Line
-	6550 5800 7250 5800
+P 7600 4800
+F 0 "U?" H 7600 5300 50  0000 C CNN
+F 1 "LTC4412xS6" H 7650 5400 50  0000 C CNN
+F 2 "Package_TO_SOT_SMD:TSOT-23-6" H 8250 4450 50  0001 C CNN
+F 3 "https://www.analog.com/media/en/technical-documentation/data-sheets/4412fb.pdf" H 9700 4600 50  0001 C CNN
+	1    7600 4800
+	1    0    0    -1
+$EndComp
 $Comp
 L power:GND #PWR?
 U 1 1 61FED494
-P 7650 6300
-F 0 "#PWR?" H 7650 6050 50  0001 C CNN
-F 1 "GND" H 7655 6127 50  0000 C CNN
-F 2 "" H 7650 6300 50  0001 C CNN
-F 3 "" H 7650 6300 50  0001 C CNN
-	1    7650 6300
-	1    0    0    -1
-$EndComp
+P 7600 5200
+F 0 "#PWR?" H 7600 4950 50  0001 C CNN
+F 1 "GND" H 7605 5027 50  0000 C CNN
+F 2 "" H 7600 5200 50  0001 C CNN
+F 3 "" H 7600 5200 50  0001 C CNN
+	1    7600 5200
+	1    0    0    -1
+$EndComp
+$Comp
+L iclr:CSD25485F5T Q?
+U 1 1 61FF0F0D
+P 8300 700
+F 0 "Q?" V 8867 800 50  0000 C CNN
+F 1 "CSD25485F5T" V 8776 800 50  0000 C CNN
+F 2 "CSD13385F5" H 8750 650 50  0001 L CNN
+F 3 "http://www.ti.com/lit/gpn/CSD25485F5" H 8750 550 50  0001 L CNN
+F 4 "-20V, P ch NexFET MOSFET, single LGA 0.8x1.5, 42mOhm" H 8750 450 50  0001 L CNN "Description"
+F 5 "0" H 8750 350 50  0001 L CNN "Height"
+F 6 "Texas Instruments" H 8750 250 50  0001 L CNN "Manufacturer_Name"
+F 7 "CSD25485F5T" H 8750 150 50  0001 L CNN "Manufacturer_Part_Number"
+F 8 "595-CSD25485F5T" H 8750 50  50  0001 L CNN "Mouser Part Number"
+F 9 "https://www.mouser.co.uk/ProductDetail/Texas-Instruments/CSD25485F5T?qs=Bho%2FbeBaDExWIlvMtFx97A%3D%3D" H 8750 -50 50  0001 L CNN "Mouser Price/Stock"
+F 10 "CSD25485F5T" H 8750 -150 50  0001 L CNN "Arrow Part Number"
+F 11 "https://www.arrow.com/en/products/csd25485f5t/texas-instruments" H 8750 -250 50  0001 L CNN "Arrow Price/Stock"
+	1    8300 700
+	0    1    1    0
+$EndComp
+Wire Wire Line
+	7500 1000 8100 1000
+Connection ~ 7500 1000
+Wire Wire Line
+	7900 1450 7900 700
+Wire Wire Line
+	7900 700  8300 700
+Wire Wire Line
+	8700 1000 10150 1000
+$Comp
+L iclr:CSD25485F5T Q?
+U 1 1 6200D1F2
+P 8350 5500
+F 0 "Q?" V 8917 5600 50  0000 C CNN
+F 1 "CSD25485F5T" V 8826 5600 50  0000 C CNN
+F 2 "CSD13385F5" H 8800 5450 50  0001 L CNN
+F 3 "http://www.ti.com/lit/gpn/CSD25485F5" H 8800 5350 50  0001 L CNN
+F 4 "-20V, P ch NexFET MOSFET, single LGA 0.8x1.5, 42mOhm" H 8800 5250 50  0001 L CNN "Description"
+F 5 "0" H 8800 5150 50  0001 L CNN "Height"
+F 6 "Texas Instruments" H 8800 5050 50  0001 L CNN "Manufacturer_Name"
+F 7 "CSD25485F5T" H 8800 4950 50  0001 L CNN "Manufacturer_Part_Number"
+F 8 "595-CSD25485F5T" H 8800 4850 50  0001 L CNN "Mouser Part Number"
+F 9 "https://www.mouser.co.uk/ProductDetail/Texas-Instruments/CSD25485F5T?qs=Bho%2FbeBaDExWIlvMtFx97A%3D%3D" H 8800 4750 50  0001 L CNN "Mouser Price/Stock"
+F 10 "CSD25485F5T" H 8800 4650 50  0001 L CNN "Arrow Part Number"
+F 11 "https://www.arrow.com/en/products/csd25485f5t/texas-instruments" H 8800 4550 50  0001 L CNN "Arrow Price/Stock"
+	1    8350 5500
+	0    1    1    0
+$EndComp
+Wire Wire Line
+	7000 4700 7200 4700
+Connection ~ 6550 5800
+$Comp
+L Device:CP_Small C?
+U 1 1 62034006
+P 6900 4700
+F 0 "C?" V 6675 4700 50  0000 C CNN
+F 1 "0.1µF" V 6766 4700 50  0000 C CNN
+F 2 "" H 6900 4700 50  0001 C CNN
+F 3 "~" H 6900 4700 50  0001 C CNN
+	1    6900 4700
+	0    1    1    0
+$EndComp
+Connection ~ 7000 4700
+$Comp
+L power:GND #PWR?
+U 1 1 620344B1
+P 6800 4700
+F 0 "#PWR?" H 6800 4450 50  0001 C CNN
+F 1 "GND" V 6805 4572 50  0000 R CNN
+F 2 "" H 6800 4700 50  0001 C CNN
+F 3 "" H 6800 4700 50  0001 C CNN
+	1    6800 4700
+	0    1    1    0
+$EndComp
+Text HLabel 8300 1950 2    50   Input ~ 0
+STAT1
+Text HLabel 8000 4900 2    50   Input ~ 0
+STAT2
+Wire Wire Line
+	6550 5800 7000 5800
+Wire Wire Line
+	7000 4700 7000 5800
+Connection ~ 7000 5800
+Wire Wire Line
+	7000 5800 8150 5800
+Wire Wire Line
+	8350 4400 8350 5500
+Wire Wire Line
+	7600 4400 8350 4400
+Wire Wire Line
+	8750 5800 10150 5800
+Wire Wire Line
+	10150 5800 10150 3700
+Connection ~ 10150 3700
 $EndSCHEMATC
