File: Powerboard/power_new_25012022.kicad_sch (KiCad schematic)
At the start: 30 parts

Commit message: usb --> uart connection added
Parts:
- removed C? (x4): C_Small, symbol Device:C_Small
- removed D?: SP0503BAHT, Package_TO_SOT_SMD:SOT-143, symbol Power_Protection:SP0503BAHT
- removed IC?: CP2102, QFN50P500X500X100-29N-D, symbol iclr:CP2102
- removed J?: USB_C_Receptacle_USB2.0, symbol Connector:USB_C_Receptacle_USB2.0
- removed Q? (x2): SI7315DN-T1-GE3, SI7315DNT1GE3, symbol iclr:SI7315DN-T1-GE3
- removed R? (x5): R_Small, symbol Device:R_Small
- added D? (x2): LED, symbol Device:LED
- added Q? (x2): SI7617DN-T1-GE3, SIS862DNT1GE3, symbol iclr:SI7617DN-T1-GE3
- added Q? (x2): MMDT2222A, Package_TO_SOT_SMD:SOT-363_SC-70-6, symbol Transistor_BJT:MMDT2222A
- added R? (x2): R_Small, symbol Device:R_Small
- added R? (x2): 10k, symbol Device:R_Small
- added TP? (x2): TestPoint, symbol Connector:TestPoint
Connections:
- net +24V: now also Q?.1 (S_1), Q?.2 (S_2), Q?.3 (S_3)
- net +3V3: now also R?.2, R?.2
- net DTR: now also Q?.4 (E2), R?.2
- net RTS: now also Q?.1 (E1), R?.2
- net RXD: now also D?.1 (K); no longer U?.41 (U0TXD/IO1)
- net TXD: now also U?.41 (U0TXD/IO1), D?.1 (K)
- net BOOT: now reaches U?.23 (IO0)
- net BOOT: now also Q?.3 (C2)
- net EN: now reaches U?.9 (EN)
- net EN: now also Q?.6 (C1), TP?.1
- net at J?.3 (Pin_3), U?.6 (SENSE): now also Q?.1 (S_1), Q?.2 (S_2), Q?.3 (S_3)
- net at U?.5 (GATE): now also Q?.4 (G), Q?.4 (G)
- new net: Q?.5 (D_1), Q?.5 (D_1), Q?.6 (D_2), Q?.6 (D_2), Q?.7 (D_3), Q?.7 (D_3), Q?.8 (D_4), Q?.8 (D_4)
- new net: D?.2 (A), R?.1 (x2)
- new net: Q?.5 (B2), R?.1
- new net: Q?.2 (B1), R?.1
- no-connect marks 21 -> 2
Other:
- added sheet USB --> UART (untitled.kicad_sch)
- moved on the sheet: C?, J?, TP?, U?
