File: Powerboard/powerboard_sc21_as25.kicad_pcb (KiCad board)
At the start: 4 copper layers, 86.1 x 55.6 mm, 172 parts, among them IC1 BQ24618RGET-iclr, IC2 CP2102, J1 Thermistor Connection 103AT N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, J10 Conn_01x04_Male, J2 Conn_01x02_Male, J3 Conn_01x02_Male, J4 Conn_01x08_Male, J5 Conn_01x04_Male, J6 Conn_01x02_Male, J7 IsolationSwitch, J8 USB_C_Receptacle_USB2.0, J9 Conn_Coaxial, Q1 RSJ250P10TL, Q10 MCH6351, Q2 RSJ250P10TL, Q3 RSJ250P10TL, Q4 RS1G120MN, Q5 RS1G120MN, Q6 MMDT2222A, Q7 RSJ250P10TL, Q8 RSJ250P10TL, Q9 MCH6351, U1 LTC4412xS6, U11 LTC4411, U2 SN65HVD230, U3 ESP32-PICO-D4, U4 RT9025-25GSP, U6 LM2679T-3.3-iclr, U7 LM2679T-3.3-iclr, U8 LTC4412xS6, U9 LTC4412xS6

Commit message: started routing, mess at the moment
Parts:
- C17, C18, C2, C22, C24, IC2, J9, R11, R4, R6, R8, TP24, U3: moved to B.Cu
- moved TP24 81.0 mm to (61.1, 53.9)
- moved C51 80.9 mm to (51.4, 72.3)
- moved C53 80.9 mm to (52.9, 72.3)
- moved C50 79.4 mm to (49.9, 72.3)
- moved IC2 78.2 mm to (53.3, 67.2)
- moved C52 76.5 mm to (54.3, 72.3)
- moved R40 74.4 mm to (51.3, 61.9)
- moved R39 74.4 mm to (52.8, 61.9)
- moved R38 74.4 mm to (54.3, 61.9)
- moved J8 74.2 mm to (55.0, 58.0), turned to 90 degrees
- moved R36 69.0 mm to (58.6, 52.4), turned to 180 degrees
- moved R35 68.2 mm to (58.5, 54.7), turned to 180 degrees
- moved R19 67.5 mm to (59.1, 69.5), turned to 180 degrees
- moved TP25 67.4 mm to (58.3, 63.0), turned to 0 degrees
- moved D2 66.9 mm to (59.1, 67.8), turned to 0 degrees
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Connections:
- C38 pad 1: Net-(C37-Pad2) -> Net-(C38-Pad1)
- C40 pad 1: Net-(C37-Pad2) -> Net-(C38-Pad1)
- C44 pad 1: Net-(C37-Pad2) -> Net-(C38-Pad1)
- C48 pad 1: Net-(C37-Pad2) -> Net-(C38-Pad1)
- J6 pad 1: Net-(C31-Pad1) -> GND
- J6 pad 2: GND -> Net-(C31-Pad1)
- J8 pad A6: Net-(D8-Pad3) -> Net-(D8-Pad4)
- J8 pad B6: Net-(D8-Pad3) -> Net-(D8-Pad4)
- L4 pad 2: Net-(C37-Pad2) -> Net-(C38-Pad1)
- Q10 pad 4: Net-(C37-Pad2) -> Net-(C38-Pad1)
- R5 pad 2: /Battery Charger/ISET2 -> /Battery Charger/ICSET2
- RPre1 pad 1: /Battery Charger/ISET2 -> /Battery Charger/ICSET2
- TP24 pad 1: Net-(D8-Pad3) -> Net-(D8-Pad4)
- U7 pad 6: Net-(C37-Pad2) -> Net-(C38-Pad1)
- U8 pad 1: Net-(C37-Pad2) -> Net-(C38-Pad1)
Routing:
- net Net-(C31-Pad1): track 2.03 -> 31.0 mm
- net VBUS: track 0.00 -> 24.6 mm
- net Net-(IC2-Pad8): track 0.00 -> 12.0 mm
- net /CANL: track 0.00 -> 11.4 mm
- net Net-(C26-Pad1): track 0.00 -> 11.2 mm
- net /CANH: track 0.00 -> 11.2 mm
- net /RTS: track 0.00 -> 11.0 mm
- net +3V3: track 0.00 -> 10.7 mm
- net Net-(J8-PadB5): track 0.00 -> 10.6 mm
- net /DTR: track 0.00 -> 8.30 mm
- net Net-(IC2-Pad9): track 0.00 -> 6.64 mm
- net /TXD: track 0.00 -> 6.06 mm
- net Net-(J8-PadA5): track 0.00 -> 3.40 mm
- net Net-(C21-Pad2): track 0.00 -> 3.11 mm
- net Net-(Q6-Pad5): track 0.00 -> 2.96 mm
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