File: Powerboard/usb__uart.kicad_sch (KiCad schematic)
At the start: 24 parts, among them IC2 CP2102, J8 USB_C_Receptacle_USB2.0, U11 LTC4411, U4 RT9025-25GSP

Commit message: layout progress
Connections:
- net at D8.3 (K), IC2.5 (D-), J8.A7 (D-)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: no longer J8.A6 (D+), J8.B6 (D+), TP24.1
- net at D8.4 (K), IC2.4 (D+): now also J8.A6 (D+), J8.B6 (D+), TP24.1
Changed lines of the file:
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@@
   (junction (at 147.32 120.65) (diameter 0) (color 0 0 0 0)
   )
+  (junction (at 124.46 96.52) (diameter 0) (color 0 0 0 0)
+  )
   (junction (at 96.52 91.44) (diameter 0) (color 0 0 0 0)
   )
   (junction (at 100.33 91.44) (diameter 0) (color 0 0 0 0)
   )
+  (junction (at 100.33 96.52) (diameter 0) (color 0 0 0 0)
+  )
   (junction (at 115.57 58.42) (diameter 0) (color 0 0 0 0)
   )
@@
   (junction (at 96.52 96.52) (diameter 0) (color 0 0 0 0)
   )
-  (junction (at 100.33 96.52) (diameter 0) (color 0 0 0 0)
-  )
   (junction (at 191.77 121.92) (diameter 0) (color 0 0 0 0)
   )
@@
   )
   (junction (at 127 54.61) (diameter 0) (color 0 0 0 0)
-  )
-  (junction (at 121.92 96.52) (diameter 0) (color 0 0 0 0)
   )
   (junction (at 134.62 62.23) (diameter 0) (color 0 0 0 0)
@@
     (stroke (width 0) (type default) (color 0 0 0 0))
   )
-  (wire (pts (xy 100.33 96.52) (xy 121.92 96.52))
-    (stroke (width 0) (type default) (color 0 0 0 0))
-  )
   (wire (pts (xy 270.51 121.92) (xy 274.32 121.92))
     (stroke (width 0) (type default) (color 0 0 0 0))
@@
     (stroke (width 0) (type default) (color 0 0 0 0))
   )
+  (wire (pts (xy 124.46 96.52) (xy 124.46 123.19))
+    (stroke (width 0) (type default) (color 0 0 0 0))
+  )
   (wire (pts (xy 111.76 78.74) (xy 114.3 78.74))
     (stroke (width 0) (type default) (color 0 0 0 0))
@@
     (stroke (width 0) (type default) (color 0 0 0 0))
   )
-  (wire (pts (xy 121.92 96.52) (xy 121.92 123.19))
-    (stroke (width 0) (type default) (color 0 0 0 0))
-  )
   (wire (pts (xy 227.33 128.27) (xy 227.33 130.81))
     (stroke (width 0) (type default) (color 0 0 0 0))
@@
     (stroke (width 0) (type default) (color 0 0 0 0))
   )
+  (wire (pts (xy 100.33 96.52) (xy 124.46 96.52))
+    (stroke (width 0) (type default) (color 0 0 0 0))
+  )
   (wire (pts (xy 215.9 121.92) (xy 227.33 121.92))
     (stroke (width 0) (type default) (color 0 0 0 0))
   )
-  (wire (pts (xy 124.46 88.9) (xy 124.46 123.19))
+  (wire (pts (xy 124.46 88.9) (xy 124.46 96.52))
     (stroke (width 0) (type default) (color 0 0 0 0))
   )
@@
     (stroke (width 0) (type default) (color 0 0 0 0))
   )
-  (wire (pts (xy 121.92 91.44) (xy 121.92 96.52))
-    (stroke (width 0) (type default) (color 0 0 0 0))
-  )
+  (wire (pts (xy 121.92 91.44) (xy 121.92 123.19))
+    (stroke (width 0) (type default) (color 0 0 0 0))
+  )
