File: Powerboard/usb__uart.kicad_sch (KiCad schematic)
At the start: 24 parts, among them IC2 CP2102, J8 USB_C_Receptacle_USB2.0, U11 LTC4411, U4 SC4216H

Commit message: update
Parts:
- C50: value 1.0uF -> 1.0muF
- C51, C53: value 0.1uF -> 0.1muF
- C52: value 4.7uF -> 4.7muF
- R37: value 470 -> 470Ω
- U4: value SC4216H -> RT9025-25GSP
Connections:
- net D+: no longer names the net of D8.3 (K), IC2.5 (D-), J8.A7 (D-), J8.B7 (D-), TP23.1
- net D+: no longer D8.4 (K), IC2.4 (D+), J8.A6 (D+), J8.B6 (D+), TP24.1
- new net: D8.4 (K), IC2.4 (D+), J8.A6 (D+), J8.B6 (D+), TP24.1
Changed lines of the file:
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@@
   (junction (at 134.62 62.23) (diameter 0) (color 0 0 0 0)
   )
-  (junction (at 76.2 116.84) (diameter 0) (color 0 0 0 0)
-  )
   (junction (at 127 62.23) (diameter 0) (color 0 0 0 0)
   )
@@
   )
   (junction (at 101.6 85.09) (diameter 0) (color 0 0 0 0)
+  )
+  (junction (at 121.92 91.44) (diameter 0) (color 0 0 0 0)
   )
   (junction (at 187.96 121.92) (diameter 0) (color 0 0 0 0)
@@
     (stroke (width 0) (type default) (color 0 0 0 0))
   )
+  (wire (pts (xy 80.01 116.84) (xy 80.01 118.7196))
+    (stroke (width 0) (type default) (color 0 0 0 0))
+  )
   (wire (pts (xy 238.76 121.92) (xy 247.65 121.92))
     (stroke (width 0) (type default) (color 0 0 0 0))
@@
     (stroke (width 0) (type default) (color 0 0 0 0))
   )
-  (wire (pts (xy 76.2 116.84) (xy 80.01 116.84))
+  (wire (pts (xy 124.46 88.9) (xy 139.7 88.9))
     (stroke (width 0) (type default) (color 0 0 0 0))
   )
@@
     (stroke (width 0) (type default) (color 0 0 0 0))
   )
+  (wire (pts (xy 100.33 91.44) (xy 121.92 91.44))
+    (stroke (width 0) (type default) (color 0 0 0 0))
+  )
   (wire (pts (xy 129.54 62.23) (xy 129.54 54.61))
     (stroke (width 0) (type default) (color 0 0 0 0))
@@
     (stroke (width 0) (type default) (color 0 0 0 0))
   )
+  (wire (pts (xy 72.39 116.84) (xy 72.39 118.872))
+    (stroke (width 0) (type default) (color 0 0 0 0))
+  )
   (wire (pts (xy 215.9 121.92) (xy 227.33 121.92))
     (stroke (width 0) (type default) (color 0 0 0 0))
@@
     (stroke (width 0) (type default) (color 0 0 0 0))
   )
+  (wire (pts (xy 121.92 91.44) (xy 139.7 91.44))
+    (stroke (width 0) (type default) (color 0 0 0 0))
+  )
   (wire (pts (xy 115.57 58.42) (xy 115.57 62.23))
     (stroke (width 0) (type default) (color 0 0 0 0))
@@
   (wire (pts (xy 95.25 91.44) (xy 96.52 91.44))
     (stroke (width 0) (type default) (color 0 0 0 0))
-  )
-  (wire (pts (xy 72.39 116.84) (xy 76.2 116.84))
-    (stroke (width 0) (type default) (color 0 0 0 0))
-  )
-  (label "D-" (at 124.46 123.19 90)
-    (effects (font (size 1.27 1.27)) (justify left bottom))
-  )
-  (label "D-" (at 96.52 91.44 0)
-    (effects (font (size 1.27 1.27)) (justify left bottom))
-  )
-  (label "D-" (at 139.7 91.44 180)
-    (effects (font (size 1.27 1.27)) (justify right bottom))
-  )
-  (label "D+" (at 96.52 96.52 0)
-    (effects (font (size 1.27 1.27)) (justify left bottom))
-  )
-  (label "D+" (at 121.92 123.19 90)
-    (effects (font (size 1.27 1.27)) (justify left bottom))
-  )
-  (label "D+" (at 139.7 88.9 180)
-    (effects (font (size 1.27 1.27)) (justify right bottom))
   )
   (label "VBUS" (at 119.38 123.19 90)
@@
     (in_bom yes) (on_board yes) (fields_autoplaced)
     (property "Reference" "U4" (id 0) (at 205.74 115.8072 0))
-    (property "Value" "SC4216H" (id 1) (at 205.74 118.3441 0))
+    (property "Value" "RT9025-25GSP" (id 1) (at 205.74 118.3441 0))
     (property "Footprint" "iclr:SOIC127P599X175-9N" (id 2) (at 205.74 115.57 0)
       (effects (font (size 1.27 1.27)) hide)
@@
     (in_bom yes) (on_board yes)
     (property "Reference" "C50" (id 0) (at 121.92 52.07 90))
-    (property "Value" "1.0uF" (id 1) (at 121.92 57.15 90))
+    (property "Value" "1.0muF" (id 1) (at 121.92 57.15 90))
     (property "Footprint" "Capacitor_SMD:C_0603_1608Metric" (id 2) (at 121.92 54.61 0)
       (effects (font (size 1.27 1.27)) hide)
@@
     (in_bom yes) (on_board yes)
     (property "Reference" "C53" (id 0) (at 132.08 59.69 90))
-    (property "Value" "0.1uF" (id 1) (at 132.08 64.77 90))
+    (property "Value" "0.1muF" (id 1) (at 132.08 64.77 90))
     (property "Footprint" "Capacitor_SMD:C_0603_1608Metric" (id 2) (at 132.08 62.23 0)
       (effects (font (size 1.27 1.27)) hide)
@@
     (in_bom yes) (on_board yes)
     (property "Reference" "C51" (id 0) (at 121.92 59.69 90))
-    (property "Value" "0.1uF" (id 1) (at 121.92 64.77 90))
+    (property "Value" "0.1muF" (id 1) (at 121.92 64.77 90))
     (property "Footprint" "Capacitor_SMD:C_0603_1608Metric" (id 2) (at 121.92 62.23 0)
       (effects (font (size 1.27 1.27)) hide)
@@
     (in_bom yes) (on_board yes)
     (property "Reference" "C52" (id 0) (at 132.08 52.07 90))
-    (property "Value" "4.7uF" (id 1) (at 132.08 57.15 90))
+    (property "Value" "4.7muF" (id 1) (at 132.08 57.15 90))
     (property "Footprint" "Capacitor_SMD:C_0603_1608Metric" (id 2) (at 132.08 54.61 0)
       (effects (font (size 1.27 1.27)) hide)
@@
   (symbol (lib_id "Device:R_Small") (at 101.6 78.74 90) (unit 1)
     (in_bom yes) (on_board yes)
-    (property "Reference" "R37" (id 0) (at 101.6 73.66 90))
-    (property "Value" "470" (id 1) (at 101.6 76.2 90))
+    (property "Reference" "R37" (id 0) (at 101.6 77.47 90))
+    (property "Value" "470Ω" (id 1) (at 101.6 80.01 90))
     (property "Footprint" "Resistor_SMD:R_0603_1608Metric" (id 2) (at 101.6 78.74 0)
       (effects (font (size 1.27 1.27)) hide)
@@
     )
     (property "Datasheet" "" (id 3) (at 147.32 133.35 0)
+      (effects (font (size 1.27 1.27)) hide)
+    )
+    (pin "1")
+  )
+  (symbol (lib_id "power:GND") (at 72.39 118.872 0) (unit 1)
+    (in_bom yes) (on_board yes)
+    (property "Reference" "#PWR0151" (id 0) (at 72.39 125.222 0)
+      (effects (font (size 1.27 1.27)) hide)
+    )
+    (property "Value" "GND" (id 1) (at 77.47 121.412 0)
+      (effects (font (size 1.27 1.27)) (justify right))
+    )
+    (property "Footprint" "" (id 2) (at 72.39 118.872 0)
+      (effects (font (size 1.27 1.27)) hide)
+    )
+    (property "Datasheet" "" (id 3) (at 72.39 118.872 0)
       (effects (font (size 1.27 1.27)) hide)
     )
@@
     (pin "9")
   )
-  (symbol (lib_id "power:GND") (at 76.2 116.84 0) (unit 1)
-    (in_bom yes) (on_board yes)
-    (property "Reference" "#PWR0150" (id 0) (at 76.2 123.19 0)
-      (effects (font (size 1.27 1.27)) hide)
-    )
-    (property "Value" "GND" (id 1) (at 81.28 119.38 0)
-      (effects (font (size 1.27 1.27)) (justify right))
-    )
-    (property "Footprint" "" (id 2) (at 76.2 116.84 0)
-      (effects (font (size 1.27 1.27)) hide)
-    )
-    (property "Datasheet" "" (id 3) (at 76.2 116.84 0)
-      (effects (font (size 1.27 1.27)) hide)
-    )
-    (pin "1")
-  )
   (symbol (lib_id "power:GND") (at 205.74 137.16 0) (unit 1)
     (in_bom yes) (on_board yes)
@@
       (effects (font (size 1.27 1.27)) hide)
     )
+    (pin "1")
+  )
+  (symbol (lib_id "power:GND") (at 80.01 118.7196 0) (unit 1)
+    (in_bom yes) (on_board yes)
+    (property "Reference" "#PWR0150" (id 0) (at 80.01 125.0696 0)
+      (effects (font (size 1.27 1.27)) hide)
+    )
+    (property "Value" "GND" (id 1) (at 85.09 121.2596 0)
+      (effects (font (size 1.27 1.27)) (justify right))
+    )
+    (property "Footprint" "" (id 2) (at 80.01 118.7196 0)
+      (effects (font (size 1.27 1.27)) hide)
+    )
+    (property "Datasheet" "" (id 3) (at 80.01 118.7196 0)
+      (effects (font (size 1.27 1.27)) hide)
+    )

Commit message: Changed some values and footprints since some went out of stock
Parts:
- C50: value 1.0muF -> 1.0uF
- C51, C53: value 0.1muF -> 0.1uF
- C52: value 4.7muF -> 4.7uF
- C54, C57: footprint Capacitor_SMD:C_0805_2012Metric -> Capacitor_SMD:C_0603_1608Metric
- R37: value 470Ω -> 470
- U4: value RT9025-25GSP -> SC4216H
Connections:
- net GND: now also IC2.29 (EPAD)
- net D-: now reaches D8.3 (K), IC2.5 (D-), J8.A7 (D-), J8.B7 (D-), TP23.1
- net D+: now reaches D8.4 (K), IC2.4 (D+), J8.A6 (D+), J8.B6 (D+), TP24.1
Changed lines of the file:
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@@
   (no_connect (at 172.72 86.36))
   (no_connect (at 152.4 63.5))
-  (no_connect (at 147.32 63.5))
+  (no_connect (at 172.72 96.52))
   (no_connect (at 95.25 106.68))
   (no_connect (at 215.9 134.62))
@@
     (stroke (width 0) (type default) (color 0 0 0 0))
   )
+  (label "D+" (at 137.16 88.9 0)
+    (effects (font (size 1.27 1.27)) (justify left bottom))
+  )
+  (label "D+" (at 97.79 96.52 0)
+    (effects (font (size 1.27 1.27)) (justify left bottom))
+  )
+  (label "D-" (at 97.79 91.44 0)
+    (effects (font (size 1.27 1.27)) (justify left bottom))
+  )
+  (label "D-" (at 137.4416 91.44 0)
+    (effects (font (size 1.27 1.27)) (justify left bottom))
+  )
+  (label "D+" (at 124.46 123.19 90)
+    (effects (font (size 1.27 1.27)) (justify left bottom))
+  )
   (label "VBUS" (at 119.38 123.19 90)
+    (effects (font (size 1.27 1.27)) (justify left bottom))
+  )
+  (label "D-" (at 121.92 123.19 90)
     (effects (font (size 1.27 1.27)) (justify left bottom))
   )
@@
       (effects (font (size 1.27 1.27)) (justify right))
     )
-    (property "Footprint" "Capacitor_SMD:C_0805_2012Metric" (id 2) (at 191.77 124.46 0)
+    (property "Footprint" "Capacitor_SMD:C_0603_1608Metric" (id 2) (at 191.77 124.46 0)
       (effects (font (size 1.27 1.27)) hide)
     )
@@
     (in_bom yes) (on_board yes) (fields_autoplaced)
     (property "Reference" "U4" (id 0) (at 205.74 115.8072 0))
-    (property "Value" "RT9025-25GSP" (id 1) (at 205.74 118.3441 0))
+    (property "Value" "SC4216H" (id 1) (at 205.74 118.3441 0))
     (property "Footprint" "iclr:SOIC127P599X175-9N" (id 2) (at 205.74 115.57 0)
       (effects (font (size 1.27 1.27)) hide)
@@
     (in_bom yes) (on_board yes)
     (property "Reference" "C50" (id 0) (at 121.92 52.07 90))
-    (property "Value" "1.0muF" (id 1) (at 121.92 57.15 90))
+    (property "Value" "1.0uF" (id 1) (at 121.92 57.15 90))
     (property "Footprint" "Capacitor_SMD:C_0603_1608Metric" (id 2) (at 121.92 54.61 0)
       (effects (font (size 1.27 1.27)) hide)
@@
     (in_bom yes) (on_board yes)
     (property "Reference" "C53" (id 0) (at 132.08 59.69 90))
-    (property "Value" "0.1muF" (id 1) (at 132.08 64.77 90))
+    (property "Value" "0.1uF" (id 1) (at 132.08 64.77 90))
     (property "Footprint" "Capacitor_SMD:C_0603_1608Metric" (id 2) (at 132.08 62.23 0)
       (effects (font (size 1.27 1.27)) hide)
@@
     (in_bom yes) (on_board yes)
     (property "Reference" "C51" (id 0) (at 121.92 59.69 90))
-    (property "Value" "0.1muF" (id 1) (at 121.92 64.77 90))
+    (property "Value" "0.1uF" (id 1) (at 121.92 64.77 90))
     (property "Footprint" "Capacitor_SMD:C_0603_1608Metric" (id 2) (at 121.92 62.23 0)
       (effects (font (size 1.27 1.27)) hide)
@@
     (in_bom yes) (on_board yes)
     (property "Reference" "C52" (id 0) (at 132.08 52.07 90))
-    (property "Value" "4.7muF" (id 1) (at 132.08 57.15 90))
+    (property "Value" "4.7uF" (id 1) (at 132.08 57.15 90))
     (property "Footprint" "Capacitor_SMD:C_0603_1608Metric" (id 2) (at 132.08 54.61 0)
       (effects (font (size 1.27 1.27)) hide)
@@
     (in_bom yes) (on_board yes)
     (property "Reference" "R37" (id 0) (at 101.6 77.47 90))
-    (property "Value" "470Ω" (id 1) (at 101.6 80.01 90))
+    (property "Value" "470" (id 1) (at 101.6 80.01 90))
     (property "Footprint" "Resistor_SMD:R_0603_1608Metric" (id 2) (at 101.6 78.74 0)
       (effects (font (size 1.27 1.27)) hide)
@@
       (effects (font (size 1.27 1.27)) (justify right))
     )
-    (property "Footprint" "Capacitor_SMD:C_0805_2012Metric" (id 2) (at 238.76 124.46 0)
+    (property "Footprint" "Capacitor_SMD:C_0603_1608Metric" (id 2) (at 238.76 124.46 0)
       (effects (font (size 1.27 1.27)) hide)
     )
@@
     (pin "2")
   )
+  (symbol (lib_id "power:GND") (at 147.32 63.5 180) (unit 1)
+    (in_bom yes) (on_board yes)
+    (property "Reference" "#PWR0173" (id 0) (at 147.32 57.15 0)
+      (effects (font (size 1.27 1.27)) hide)
+    )
+    (property "Value" "GND" (id 1) (at 142.24 60.96 0)
+      (effects (font (size 1.27 1.27)) (justify right))
+    )
+    (property "Footprint" "" (id 2) (at 147.32 63.5 0)
+      (effects (font (size 1.27 1.27)) hide)
+    )
+    (property "Datasheet" "" (id 3) (at 147.32 63.5 0)
+      (effects (font (size 1.27 1.27)) hide)
+    )
+    (pin "1")
+  )
   (symbol (lib_id "Device:R_Small") (at 97.79 83.82 270) (unit 1)
