File: Powerboard/battchrg.kicad_sch (KiCad schematic)
At the start: 61 parts, among them IC1 BQ24618RGET-iclr, J1 Thermistor Connection 103AT N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, J5 Conn_01x04_Male, J6 Conn_01x02_Male, J7 IsolationSwitch, Q1 RSJ250P10TL, Q2 RSJ250P10TL, Q3 RSJ250P10TL, Q4 RS1G120MN, Q5 RS1G120MN

Commit message: update
Parts:
- removed RAC1: 10m, Resistor_SMD:R_0603_1608Metric, symbol Device:R_Small
- removed TP16, TP17, TP18: TestPoint, TestPoint:TestPoint_Pad_D1.0mm, symbol Connector:TestPoint
- C1, C10, C11, C3, C31, C33: value 0.1uF -> 0.1μF
- C14, C15, C6: value 0.1uF -> 0.1µF
- C32: value 22uF -> 22μF; footprint Capacitor_SMD:C_1206_3216Metric -> Capacitor_SMD:C_1210_3225Metric
- C4: value 1uF -> 1μF
- L1: value 6.8uH -> 6.8µH
- R1: value 10k -> 10kΩ
- R10: value 430k -> 430kΩ
- R14, R15, R3, R5, R7: value 100k -> 100kΩ
- R16: value 100 -> 100Ω
- R17: value 10 -> 10Ω
- R18, R32: value 1k -> 1kΩ
- R2: value 110k -> 110kΩ
- R20: value 2 -> 2Ω
- R28, R29: value 3k -> 3.5k
- R9: value 9.31k -> 9.31kΩ
- RAdp1: value 150k -> 150kΩ
- RFast1: value 32k -> 32kΩ
- RPre1: value 13k -> 13kΩ
- RSR1: value 10m -> 10mΩ
Connections:
- net at PowerLED1.2 (A), Q1.3, R20.2: now also J5.1 (Pin_1), J5.2 (Pin_2)

Commit message: Changed some values and footprints since some went out of stock
Parts:
- C1, C10, C11, C3, C31, C33: value 0.1μF -> 0.1uF
- C14, C15, C6: value 0.1µF -> 0.1uF
- C32: value 22μF -> 22uF; footprint Capacitor_SMD:C_1210_3225Metric -> Capacitor_SMD:C_1206_3216Metric
- C4: value 1μF -> 1uF
- L1: value 6.8µH -> 6.8uH
- R1: value 10kΩ -> 10k
- R10: value 430kΩ -> 430k
- R14, R15, R3, R5, R7: value 100kΩ -> 100k
- R16: value 100Ω -> 100
- R17: value 10Ω -> 10
- R18, R32: value 1kΩ -> 1k
- R2: value 110kΩ -> 110k
- R20: value 2Ω -> 2
- R28, R29: value 3.5k -> 3k
- R9: value 9.31kΩ -> 9.31k
- RAC1: footprint RESC50110X50N -> (none)
- RAdp1: value 150kΩ -> 150k
- RFast1: value 32kΩ -> 32k
- RPre1: value 13kΩ -> 13k
- RSR1: value 10mΩ -> 10m
Changed lines of the file:
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@@
     (in_bom yes) (on_board yes)
     (property "Reference" "R16" (id 0) (at 191.77 119.38 90))
-    (property "Value" "100Ω" (id 1) (at 191.77 121.92 90))
+    (property "Value" "100" (id 1) (at 191.77 121.92 90))
     (property "Footprint" "Resistor_SMD:R_0603_1608Metric" (id 2) (at 189.23 118.11 0)
       (effects (font (size 1.27 1.27)) hide)
@@
       (effects (font (size 1.27 1.27)) (justify right))
     )
-    (property "Value" "430kΩ" (id 1) (at 184.15 125.73 0)
+    (property "Value" "430k" (id 1) (at 184.15 125.73 0)
       (effects (font (size 1.27 1.27)) (justify right))
     )
@@
       (effects (font (size 1.27 1.27)) (justify right))
     )
-    (property "Value" "9.31kΩ" (id 1) (at 184.15 115.57 0)
+    (property "Value" "9.31k" (id 1) (at 184.15 115.57 0)
       (effects (font (size 1.27 1.27)) (justify right))
     )
@@
       (effects (font (size 1.27 1.27)) (justify left))
     )
-    (property "Value" "0.1μF" (id 1) (at 199.1868 123.063 0)
+    (property "Value" "0.1uF" (id 1) (at 199.1868 123.063 0)
       (effects (font (size 1.27 1.27)) (justify left))
     )
@@
       (effects (font (size 1.27 1.27)) (justify left))
     )
-    (property "Value" "100kΩ" (id 1) (at 233.68 137.16 0)
+    (property "Value" "100k" (id 1) (at 233.68 137.16 0)
       (effects (font (size 1.27 1.27)) (justify left))
     )
@@
       (effects (font (size 1.27 1.27)) (justify left))
     )
-    (property "Value" "100kΩ" (id 1) (at 248.92 137.16 0)
+    (property "Value" "100k" (id 1) (at 248.92 137.16 0)
       (effects (font (size 1.27 1.27)) (justify left))
     )
@@
       (effects (font (size 1.27 1.27)) (justify left))
     )
-    (property "Value" "100kΩ" (id 1) (at 242.57 137.16 0)
+    (property "Value" "100k" (id 1) (at 242.57 137.16 0)
       (effects (font (size 1.27 1.27)) (justify left))
     )
@@
       (effects (font (size 1.27 1.27)) (justify left))
     )
-    (property "Value" "32kΩ" (id 1) (at 234.95 152.4 0)
+    (property "Value" "32k" (id 1) (at 234.95 152.4 0)
       (effects (font (size 1.27 1.27)) (justify left))
     )
@@
       (effects (font (size 1.27 1.27)) (justify left))
     )
-    (property "Value" "150kΩ" (id 1) (at 248.92 152.4 0)
+    (property "Value" "150k" (id 1) (at 248.92 152.4 0)
       (effects (font (size 1.27 1.27)) (justify left))
     )
@@
       (effects (font (size 1.27 1.27)) (justify left))
     )
-    (property "Value" "13kΩ" (id 1) (at 242.57 152.4 0)
+    (property "Value" "13k" (id 1) (at 242.57 152.4 0)
       (effects (font (size 1.27 1.27)) (justify left))
     )
@@
       (effects (font (size 1.27 1.27)) (justify left))
     )
-    (property "Value" "0.1μF" (id 1) (at 200.914 95.504 90)
+    (property "Value" "0.1uF" (id 1) (at 200.914 95.504 90)
       (effects (font (size 1.27 1.27)) (justify left))
     )
@@
       (effects (font (size 1.27 1.27)) (justify left))
     )
-    (property "Value" "100kΩ" (id 1) (at 147.32 115.57 90)
+    (property "Value" "100k" (id 1) (at 147.32 115.57 90)
       (effects (font (size 1.27 1.27)) (justify left))
     )
@@
       (effects (font (size 1.27 1.27)) (justify left))
     )
-    (property "Value" "0.1µF" (id 1) (at 144.78 107.95 90)
+    (property "Value" "0.1uF" (id 1) (at 144.78 107.95 90)
       (effects (font (size 1.27 1.27)) (justify left))
     )
@@
       (effects (font (size 1.27 1.27)) (justify left))
     )
-    (property "Value" "10Ω" (id 1) (at 133.35 110.49 90)
+    (property "Value" "10" (id 1) (at 133.35 110.49 90)
       (effects (font (size 1.27 1.27)) (justify left))
     )
@@
     (in_bom yes) (on_board yes)
     (property "Reference" "R18" (id 0) (at 157.48 102.9716 90))
-    (property "Value" "1kΩ" (id 1) (at 157.48 105.283 90))
+    (property "Value" "1k" (id 1) (at 157.48 105.283 90))
     (property "Footprint" "Resistor_SMD:R_0603_1608Metric" (id 2) (at 157.48 107.95 0)
       (effects (font (size 1.27 1.27)) hide)
@@
       (effects (font (size 1.27 1.27)) (justify left))
     )
-    (property "Value" "0.1μF" (id 1) (at 254 114.3 0)
+    (property "Value" "0.1uF" (id 1) (at 254 114.3 0)
       (effects (font (size 1.27 1.27)) (justify left))
     )
@@
       (effects (font (size 1.27 1.27)) (justify left))
     )
-    (property "Value" "0.1μF" (id 1) (at 246.38 121.92 0)
+    (property "Value" "0.1uF" (id 1) (at 246.38 121.92 0)
       (effects (font (size 1.27 1.27)) (justify left))
     )
@@
       (effects (font (size 1.27 1.27)) (justify left))
     )
-    (property "Value" "100kΩ" (id 1) (at 199.39 62.23 90)
+    (property "Value" "100k" (id 1) (at 199.39 62.23 90)
       (effects (font (size 1.27 1.27)) (justify left))
     )
@@
       (effects (font (size 1.27 1.27)) (justify left))
     )
-    (property "Value" "0.1µF" (id 1) (at 204.47 68.58 90)
+    (property "Value" "0.1uF" (id 1) (at 204.47 68.58 90)
       (effects (font (size 1.27 1.27)) (justify left))
     )
@@
       (effects (font (size 1.27 1.27)) (justify left))
     )
-    (property "Value" "0.1μF" (id 1) (at 196.85 104.14 90)
+    (property "Value" "0.1uF" (id 1) (at 196.85 104.14 90)
       (effects (font (size 1.27 1.27)) (justify left))
     )
@@
       (effects (font (size 1.27 1.27)) (justify left))
     )
-    (property "Value" "1μF" (id 1) (at 195.58 111.76 90)
+    (property "Value" "1uF" (id 1) (at 195.58 111.76 90)
       (effects (font (size 1.27 1.27)) (justify left))
     )
@@
       (effects (font (size 1.27 1.27)) (justify left))
     )
-    (property "Value" "2Ω" (id 1) (at 72.39 62.23 0)
+    (property "Value" "2" (id 1) (at 72.39 62.23 0)
       (effects (font (size 1.27 1.27)) (justify left))
     )
@@
       (effects (font (size 1.27 1.27)) (justify left))
     )
-    (property "Value" "1kΩ" (id 1) (at 214.63 73.66 0)
+    (property "Value" "1k" (id 1) (at 214.63 73.66 0)
       (effects (font (size 1.27 1.27)) (justify left))
     )
@@
     (in_bom yes) (on_board yes)
     (property "Reference" "R2" (id 0) (at 55.88 119.38 90))
-    (property "Value" "110kΩ" (id 1) (at 62.23 119.38 90))
+    (property "Value" "110k" (id 1) (at 62.23 119.38 90))
     (property "Footprint" "Resistor_SMD:R_0603_1608Metric" (id 2) (at 58.42 121.92 0)
       (effects (font (size 1.27 1.27)) hide)
@@
     (in_bom yes) (on_board yes)
     (property "Reference" "R1" (id 0) (at 45.72 124.46 90))
-    (property "Value" "10kΩ" (id 1) (at 45.72 129.54 90))
+    (property "Value" "10k" (id 1) (at 45.72 129.54 90))
     (property "Footprint" "Resistor_SMD:R_0603_1608Metric" (id 2) (at 45.72 127 0)
       (effects (font (size 1.27 1.27)) hide)
@@
       (effects (font (size 1.27 1.27)) (justify left))
     )
-    (property "Value" "10mΩ" (id 1) (at 93.1784 123.866 90)
+    (property "Value" "10m" (id 1) (at 93.1784 123.866 90)
       (effects (font (size 1.27 1.27)) (justify left))
     )
@@
       (effects (font (size 1.27 1.27)) (justify left))
     )
-    (property "Value" "6.8µH" (id 1) (at 100.33 128.27 90)
+    (property "Value" "6.8uH" (id 1) (at 100.33 128.27 90)
       (effects (font (size 1.27 1.27)) (justify left))
     )
@@
       (effects (font (size 1.27 1.27)) (justify left))
     )
-    (property "Value" "0.1µF" (id 1) (at 110.49 129.54 90)
+    (property "Value" "0.1uF" (id 1) (at 110.49 129.54 90)
       (effects (font (size 1.27 1.27)) (justify left))
     )
@@
     (in_bom yes) (on_board yes)
     (property "Reference" "C31" (id 0) (at 108.1577 184.5801 90))
-    (property "Value" "0.1μF" (id 1) (at 108.164 187.3161 90))
+    (property "Value" "0.1uF" (id 1) (at 108.164 187.3161 90))
     (property "Footprint" "Capacitor_SMD:C_0603_1608Metric" (id 2) (at 104.14 185.801 0)
       (effects (font (size 1.27 1.27)) hide)
@@
       (effects (font (size 1.27 1.27)) (justify left))
     )
-    (property "Value" "3.5k" (id 1) (at 64.77 46.99 0)
+    (property "Value" "3k" (id 1) (at 64.77 46.99 0)
       (effects (font (size 1.27 1.27)) (justify left))
     )
@@
       (effects (font (size 1.27 1.27)) (justify left))
     )
-    (property "Value" "3.5k" (id 1) (at 54.61 139.7 90)
+    (property "Value" "3k" (id 1) (at 54.61 139.7 90)
       (effects (font (size 1.27 1.27)) (justify left))
     )
@@
     (property "Reference" "RAC1" (id 0) (at 194.818 89.061 0))
     (property "Value" "FCSL110R010FER" (id 1) (at 194.818 91.5979 0))
-    (property "Footprint" "RESC50110X50N" (id 2) (at 199.898 92.71 0)
+    (property "Footprint" "" (id 2) (at 199.898 92.71 0)
       (effects (font (size 1.27 1.27)) (justify left) hide)
     )
@@
     (in_bom yes) (on_board yes)
     (property "Reference" "C32" (id 0) (at 104.394 192.786 90))
-    (property "Value" "22μF" (id 1) (at 104.267 194.818 90))
-    (property "Footprint" "Capacitor_SMD:C_1210_3225Metric" (id 2) (at 104.14 189.992 0)
-      (effects (font (size 1.27 1.27)) hide)
-    )
+    (property "Value" "22uF" (id 1) (at 104.267 194.818 90))
+    (property "Footprint" "Capacitor_SMD:C_1206_3216Metric" (id 2) (at 104.14 189.992 0)
+      (effects (font (size 1.27 1.27)) hide)
+    )

Commit message: Change RSR and RAC sense resistor to ones rated for 5W
Parts:
- removed RSR1: 10m, Resistor_SMD:R_0603_1608Metric, symbol Device:R_Small
- added RSR1: FCSL110R010FER, iclr:RESC50110X70N, symbol iclr:FCSL110R010FER
- RAC1: footprint (none) -> iclr:RESC50110X70N
Connections:
- net Q3-S: now also RSR1.1
- net SRP: now also RSR1.2
Other:
- moved on the sheet: C6, L1
Changed lines of the file:
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@@
   (junction (at 247.65 130.81) (diameter 0) (color 0 0 0 0)
   )
-  (junction (at 102.87 121.92) (diameter 0) (color 0 0 0 0)
+  (junction (at 115.57 121.92) (diameter 0) (color 0 0 0 0)
   )
   (junction (at 138.43 105.41) (diameter 0) (color 0 0 0 0)
@@
   (junction (at 63.5 127) (diameter 0) (color 0 0 0 0)
   )
-  (junction (at 102.87 127) (diameter 0) (color 0 0 0 0)
+  (junction (at 115.57 127) (diameter 0) (color 0 0 0 0)
   )
   (junction (at 247.65 143.51) (diameter 0) (color 0 0 0 0)
@@
   (junction (at 73.66 57.15) (diameter 0) (color 0 0 0 0)
   )
-  (junction (at 113.03 127) (diameter 0) (color 0 0 0 0)
+  (junction (at 125.73 127) (diameter 0) (color 0 0 0 0)
   )
   (junction (at 94.488 180.848) (diameter 0) (color 0 0 0 0)
@@
   (junction (at 205.74 66.04) (diameter 0) (color 0 0 0 0)
   )
-  (junction (at 93.98 127) (diameter 0) (color 0 0 0 0)
+  (junction (at 106.68 127) (diameter 0) (color 0 0 0 0)
   )
   (junction (at 196.85 118.11) (diameter 0) (color 0 0 0 0)
@@
     (stroke (width 0) (type default) (color 0 0 0 0))
   )
-  (wire (pts (xy 102.87 127) (xy 104.14 127))
+  (wire (pts (xy 115.57 127) (xy 116.84 127))
     (stroke (width 0) (type default) (color 0 0 0 0))
   )
@@
     (stroke (width 0) (type default) (color 0 0 0 0))
   )
-  (wire (pts (xy 113.03 127) (xy 114.3 127))
-    (stroke (width 0) (type default) (color 0 0 0 0))
-  )
-  (wire (pts (xy 100.33 121.92) (xy 102.87 121.92))
+  (wire (pts (xy 125.73 127) (xy 127 127))
+    (stroke (width 0) (type default) (color 0 0 0 0))
+  )
+  (wire (pts (xy 113.03 121.92) (xy 115.57 121.92))
     (stroke (width 0) (type default) (color 0 0 0 0))
   )
@@
     (stroke (width 0) (type default) (color 0 0 0 0))
   )
-  (wire (pts (xy 93.98 113.03) (xy 93.98 127))
+  (wire (pts (xy 106.68 113.03) (xy 106.68 127))
     (stroke (width 0) (type default) (color 0 0 0 0))
   )
@@
     (stroke (width 0) (type default) (color 0 0 0 0))
   )
-  (wire (pts (xy 92.71 127) (xy 93.98 127))
+  (wire (pts (xy 105.41 127) (xy 106.68 127))
     (stroke (width 0) (type default) (color 0 0 0 0))
   )
@@
     (stroke (width 0) (type default) (color 0 0 0 0))
   )
-  (wire (pts (xy 113.03 127) (xy 113.03 133.35))
+  (wire (pts (xy 125.73 127) (xy 125.73 133.35))
     (stroke (width 0) (type default) (color 0 0 0 0))
   )
@@
     (stroke (width 0) (type default) (color 0 0 0 0))
   )
-  (wire (pts (xy 102.87 121.92) (xy 110.49 121.92))
+  (wire (pts (xy 115.57 121.92) (xy 123.19 121.92))
     (stroke (width 0) (type default) (color 0 0 0 0))
   )
@@
     (stroke (width 0) (type default) (color 0 0 0 0))
   )
-  (wire (pts (xy 102.87 127) (xy 102.87 133.35))
+  (wire (pts (xy 115.57 127) (xy 115.57 133.35))
     (stroke (width 0) (type default) (color 0 0 0 0))
   )
@@
     (stroke (width 0) (type default) (color 0 0 0 0))
   )
-  (wire (pts (xy 102.87 121.92) (xy 102.87 127))
+  (wire (pts (xy 115.57 121.92) (xy 115.57 127))
     (stroke (width 0) (type default) (color 0 0 0 0))
   )
@@
     (stroke (width 0) (type default) (color 0 0 0 0))
   )
-  (wire (pts (xy 101.6 127) (xy 102.87 127))
+  (wire (pts (xy 114.3 127) (xy 115.57 127))
     (stroke (width 0) (type default) (color 0 0 0 0))
   )
@@
     (stroke (width 0) (type default) (color 0 0 0 0))
   )
-  (wire (pts (xy 109.22 127) (xy 113.03 127))
+  (wire (pts (xy 121.92 127) (xy 125.73 127))
     (stroke (width 0) (type default) (color 0 0 0 0))
   )
@@
     (effects (font (size 1.27 1.27)) (justify right bottom))
   )
-  (label "SRP" (at 93.98 113.03 180)
+  (label "SRP" (at 106.68 113.03 180)
     (effects (font (size 1.27 1.27)) (justify right bottom))
   )
@@
     (effects (font (size 1.27 1.27)) (justify right bottom))
   )
-  (label "PH" (at 110.49 121.92 0)
+  (label "PH" (at 123.19 121.92 0)
     (effects (font (size 1.27 1.27)) (justify left bottom))
   )
@@
     (effects (font (size 1.27 1.27)) (justify left bottom))
   )
-  (label "Q4-S" (at 100.33 121.92 180)
+  (label "Q4-S" (at 113.03 121.92 180)
     (effects (font (size 1.27 1.27)) (justify right bottom))
   )
@@
     (effects (font (size 1.27 1.27)) (justify right bottom))
   )
-  (label "BTST" (at 113.03 133.35 180)
+  (label "BTST" (at 125.73 133.35 180)
     (effects (font (size 1.27 1.27)) (justify right bottom))
   )
@@
     (effects (font (size 1.27 1.27)) (justify left bottom))
   )
-  (label "Q5-D" (at 102.87 133.35 180)
+  (label "Q5-D" (at 115.57 133.35 180)
     (effects (font (size 1.27 1.27)) (justify right bottom))
   )
@@
     (effects (font (size 1.27 1.27)) (justify left bottom))
   )
-  (label "BTSTP" (at 114.3 127 0)
+  (label "BTSTP" (at 127 127 0)
     (effects (font (size 1.27 1.27)) (justify left bottom))
   )
@@
     (pin "1")
   )
-  (symbol (lib_id "Device:R_Small") (at 90.17 127 90) (unit 1)
-    (in_bom yes) (on_board yes)
-    (property "Reference" "RSR1" (id 0) (at 91.9084 121.326 90)
-      (effects (font (size 1.27 1.27)) (justify left))
-    )
-    (property "Value" "10m" (id 1) (at 93.1784 123.866 90)
-      (effects (font (size 1.27 1.27)) (justify left))
-    )
-    (property "Footprint" "Resistor_SMD:R_0603_1608Metric" (id 2) (at 90.17 127 0)
-      (effects (font (size 1.27 1.27)) hide)
-    )
-    (property "Datasheet" "~" (id 3) (at 90.17 127 0)
-      (effects (font (size 1.27 1.27)) hide)
-    )
-    (pin "1")
-    (pin "2")
-  )
-  (symbol (lib_id "Device:L") (at 97.79 127 90) (unit 1)
-    (in_bom yes) (on_board yes)
-    (property "Reference" "L1" (id 0) (at 97.79 124.46 90)
-      (effects (font (size 1.27 1.27)) (justify left))
-    )
-    (property "Value" "6.8uH" (id 1) (at 100.33 128.27 90)
-      (effects (font (size 1.27 1.27)) (justify left))
-    )
-    (property "Footprint" "iclr:INDM8681X400N" (id 2) (at 97.79 127 0)
-      (effects (font (size 1.27 1.27)) hide)
-    )
-    (property "Datasheet" "~" (id 3) (at 97.79 127 0)
-      (effects (font (size 1.27 1.27)) hide)
-    )
-    (pin "1")
-    (pin "2")
-  )
-  (symbol (lib_id "Device:C_Small") (at 106.68 127 90) (unit 1)
-    (in_bom yes) (on_board yes)
-    (property "Reference" "C6" (id 0) (at 107.95 124.46 90)
-      (effects (font (size 1.27 1.27)) (justify left))
-    )
-    (property "Value" "0.1uF" (id 1) (at 110.49 129.54 90)
-      (effects (font (size 1.27 1.27)) (justify left))
-    )
-    (property "Footprint" "Capacitor_SMD:C_0603_1608Metric" (id 2) (at 106.68 127 0)
-      (effects (font (size 1.27 1.27)) hide)
-    )
-    (property "Datasheet" "~" (id 3) (at 106.68 127 0)
+  (symbol (lib_id "Device:L") (at 110.49 127 90) (unit 1)
+    (in_bom yes) (on_board yes)
+    (property "Reference" "L1" (id 0) (at 110.49 124.46 90)
+      (effects (font (size 1.27 1.27)) (justify left))
+    )
+    (property "Value" "6.8uH" (id 1) (at 113.03 128.27 90)
+      (effects (font (size 1.27 1.27)) (justify left))
+    )
+    (property "Footprint" "iclr:INDM8681X400N" (id 2) (at 110.49 127 0)
+      (effects (font (size 1.27 1.27)) hide)
+    )
+    (property "Datasheet" "~" (id 3) (at 110.49 127 0)
+      (effects (font (size 1.27 1.27)) hide)
+    )
+    (pin "1")
+    (pin "2")
+  )
+  (symbol (lib_id "Device:C_Small") (at 119.38 127 90) (unit 1)
+    (in_bom yes) (on_board yes)
+    (property "Reference" "C6" (id 0) (at 120.65 124.46 90)
+      (effects (font (size 1.27 1.27)) (justify left))
+    )
+    (property "Value" "0.1uF" (id 1) (at 123.19 129.54 90)
+      (effects (font (size 1.27 1.27)) (justify left))
+    )
+    (property "Footprint" "Capacitor_SMD:C_0603_1608Metric" (id 2) (at 119.38 127 0)
+      (effects (font (size 1.27 1.27)) hide)
+    )
+    (property "Datasheet" "~" (id 3) (at 119.38 127 0)
       (effects (font (size 1.27 1.27)) hide)
     )
@@
     (property "Reference" "RAC1" (id 0) (at 194.818 89.061 0))
     (property "Value" "FCSL110R010FER" (id 1) (at 194.818 91.5979 0))
-    (property "Footprint" "" (id 2) (at 199.898 92.71 0)
+    (property "Footprint" "iclr:RESC50110X70N" (id 2) (at 199.898 92.71 0)
       (effects (font (size 1.27 1.27)) (justify left) hide)
     )
@@
     )
     (pin "1")
+    (pin "2")
+  )
+  (symbol (lib_id "iclr:FCSL110R010FER") (at 87.63 127 0) (unit 1)
+    (in_bom yes) (on_board yes) (fields_autoplaced)
+    (property "Reference" "RSR1" (id 0) (at 96.52 122.081 0))
+    (property "Value" "FCSL110R010FER" (id 1) (at 96.52 124.6179 0))
+    (property "Footprint" "iclr:RESC50110X70N" (id 2) (at 101.6 125.73 0)
+      (effects (font (size 1.27 1.27)) (justify left) hide)
+    )
+    (property "Datasheet" "https://www.ohmite.com/assets/docs/res_fcsl.pdf?r=false" (id 3) (at 101.6 128.27 0)
+      (effects (font (size 1.27 1.27)) (justify left) hide)
+    )
+    (property "Description" "Arcol Ohmite 10m, 4320 Metal Foil SMD Resistor +/-1% 5W - FCSL110R010FER" (id 4) (at 101.6 130.81 0)
+      (effects (font (size 1.27 1.27)) (justify left) hide)
+    )
+    (property "Height" "0.5" (id 5) (at 101.6 133.35 0)
+      (effects (font (size 1.27 1.27)) (justify left) hide)
+    )
+    (property "Manufacturer_Name" "Ohmite" (id 6) (at 101.6 135.89 0)
+      (effects (font (size 1.27 1.27)) (justify left) hide)
+    )
+    (property "Manufacturer_Part_Number" "FCSL110R010FER" (id 7) (at 101.6 138.43 0)
+      (effects (font (size 1.27 1.27)) (justify left) hide)
+    )
+    (property "Mouser Part Number" "588-FCSL110R010FER" (id 8) (at 101.6 140.97 0)
+      (effects (font (size 1.27 1.27)) (justify left) hide)
+    )
+    (property "Mouser Price/Stock" "https://www.mouser.co.uk/ProductDetail/Ohmite/FCSL110R010FER/?qs=MhoRK8A7%252BtW%2F5XGSjsF0ww%3D%3D" (id 9) (at 101.6 143.51 0)
+      (effects (font (size 1.27 1.27)) (justify left) hide)
+    )
+    (property "Arrow Part Number" "" (id 10) (at 101.6 146.05 0)
+      (effects (font (size 1.27 1.27)) (justify left) hide)
+    )
+    (property "Arrow Price/Stock" "" (id 11) (at 101.6 148.59 0)
+      (effects (font (size 1.27 1.27)) (justify left) hide)
+    )
+    (pin "1")
