File: Powerboard/battchrg.kicad_sch (KiCad schematic)
At the start: 57 parts, among them IC1 BQ24618RGET-iclr, J1 Thermistor Connection 103AT N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, J5 Conn_01x04_Male, J6 Conn_01x02_Male, J7 IsolationSwitch, Q1 RSJ250P10TL, Q2 RSJ250P10TL, Q3 RSJ250P10TL, Q4 RS1G120MN, Q5 RS1G120MN

Commit message: changed RSR again
Parts:
- removed RSR1: FCSL110R010FER, iclr:RESC50110X70N, symbol iclr:FCSL110R010FER
- added RSR1: 10m, Resistor_SMD:R_0603_1608Metric, symbol Device:R_Small
Connections:
- net Q3-S: now also RSR1.1
- net SRP: now also RSR1.2
Other:
- moved on the sheet: C6, L1
Changed lines of the file:
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@@
   (junction (at 247.65 130.81) (diameter 0) (color 0 0 0 0)
   )
-  (junction (at 115.57 121.92) (diameter 0) (color 0 0 0 0)
+  (junction (at 102.87 121.92) (diameter 0) (color 0 0 0 0)
   )
   (junction (at 138.43 105.41) (diameter 0) (color 0 0 0 0)
@@
   (junction (at 63.5 127) (diameter 0) (color 0 0 0 0)
   )
-  (junction (at 115.57 127) (diameter 0) (color 0 0 0 0)
+  (junction (at 102.87 127) (diameter 0) (color 0 0 0 0)
   )
   (junction (at 247.65 143.51) (diameter 0) (color 0 0 0 0)
@@
   (junction (at 73.66 57.15) (diameter 0) (color 0 0 0 0)
   )
-  (junction (at 125.73 127) (diameter 0) (color 0 0 0 0)
+  (junction (at 113.03 127) (diameter 0) (color 0 0 0 0)
   )
   (junction (at 94.488 180.848) (diameter 0) (color 0 0 0 0)
@@
   (junction (at 205.74 66.04) (diameter 0) (color 0 0 0 0)
   )
-  (junction (at 106.68 127) (diameter 0) (color 0 0 0 0)
+  (junction (at 93.98 127) (diameter 0) (color 0 0 0 0)
   )
   (junction (at 196.85 118.11) (diameter 0) (color 0 0 0 0)
@@
     (stroke (width 0) (type default) (color 0 0 0 0))
   )
-  (wire (pts (xy 115.57 127) (xy 116.84 127))
+  (wire (pts (xy 102.87 127) (xy 104.14 127))
     (stroke (width 0) (type default) (color 0 0 0 0))
   )
@@
     (stroke (width 0) (type default) (color 0 0 0 0))
   )
-  (wire (pts (xy 125.73 127) (xy 127 127))
-    (stroke (width 0) (type default) (color 0 0 0 0))
-  )
-  (wire (pts (xy 113.03 121.92) (xy 115.57 121.92))
+  (wire (pts (xy 113.03 127) (xy 114.3 127))
+    (stroke (width 0) (type default) (color 0 0 0 0))
+  )
+  (wire (pts (xy 100.33 121.92) (xy 102.87 121.92))
     (stroke (width 0) (type default) (color 0 0 0 0))
   )
@@
     (stroke (width 0) (type default) (color 0 0 0 0))
   )
-  (wire (pts (xy 106.68 113.03) (xy 106.68 127))
+  (wire (pts (xy 93.98 113.03) (xy 93.98 127))
     (stroke (width 0) (type default) (color 0 0 0 0))
   )
@@
     (stroke (width 0) (type default) (color 0 0 0 0))
   )
-  (wire (pts (xy 105.41 127) (xy 106.68 127))
+  (wire (pts (xy 92.71 127) (xy 93.98 127))
     (stroke (width 0) (type default) (color 0 0 0 0))
   )
@@
     (stroke (width 0) (type default) (color 0 0 0 0))
   )
-  (wire (pts (xy 125.73 127) (xy 125.73 133.35))
+  (wire (pts (xy 113.03 127) (xy 113.03 133.35))
     (stroke (width 0) (type default) (color 0 0 0 0))
   )
@@
     (stroke (width 0) (type default) (color 0 0 0 0))
   )
-  (wire (pts (xy 115.57 121.92) (xy 123.19 121.92))
+  (wire (pts (xy 102.87 121.92) (xy 110.49 121.92))
     (stroke (width 0) (type default) (color 0 0 0 0))
   )
@@
     (stroke (width 0) (type default) (color 0 0 0 0))
   )
-  (wire (pts (xy 115.57 127) (xy 115.57 133.35))
+  (wire (pts (xy 102.87 127) (xy 102.87 133.35))
     (stroke (width 0) (type default) (color 0 0 0 0))
   )
@@
     (stroke (width 0) (type default) (color 0 0 0 0))
   )
-  (wire (pts (xy 115.57 121.92) (xy 115.57 127))
+  (wire (pts (xy 102.87 121.92) (xy 102.87 127))
     (stroke (width 0) (type default) (color 0 0 0 0))
   )
@@
     (stroke (width 0) (type default) (color 0 0 0 0))
   )
-  (wire (pts (xy 114.3 127) (xy 115.57 127))
+  (wire (pts (xy 101.6 127) (xy 102.87 127))
     (stroke (width 0) (type default) (color 0 0 0 0))
   )
@@
     (stroke (width 0) (type default) (color 0 0 0 0))
   )
-  (wire (pts (xy 121.92 127) (xy 125.73 127))
+  (wire (pts (xy 109.22 127) (xy 113.03 127))
     (stroke (width 0) (type default) (color 0 0 0 0))
   )
@@
     (effects (font (size 1.27 1.27)) (justify right bottom))
   )
-  (label "SRP" (at 106.68 113.03 180)
+  (label "SRP" (at 93.98 113.03 180)
     (effects (font (size 1.27 1.27)) (justify right bottom))
   )
@@
     (effects (font (size 1.27 1.27)) (justify right bottom))
   )
-  (label "PH" (at 123.19 121.92 0)
+  (label "PH" (at 110.49 121.92 0)
     (effects (font (size 1.27 1.27)) (justify left bottom))
   )
@@
     (effects (font (size 1.27 1.27)) (justify left bottom))
   )
-  (label "Q4-S" (at 113.03 121.92 180)
+  (label "Q4-S" (at 100.33 121.92 180)
     (effects (font (size 1.27 1.27)) (justify right bottom))
   )
@@
     (effects (font (size 1.27 1.27)) (justify right bottom))
   )
-  (label "BTST" (at 125.73 133.35 180)
+  (label "BTST" (at 113.03 133.35 180)
     (effects (font (size 1.27 1.27)) (justify right bottom))
   )
@@
     (effects (font (size 1.27 1.27)) (justify left bottom))
   )
-  (label "Q5-D" (at 115.57 133.35 180)
+  (label "Q5-D" (at 102.87 133.35 180)
     (effects (font (size 1.27 1.27)) (justify right bottom))
   )
@@
     (effects (font (size 1.27 1.27)) (justify left bottom))
   )
-  (label "BTSTP" (at 127 127 0)
+  (label "BTSTP" (at 114.3 127 0)
     (effects (font (size 1.27 1.27)) (justify left bottom))
   )
@@
     (pin "1")
   )
-  (symbol (lib_id "Device:L") (at 110.49 127 90) (unit 1)
-    (in_bom yes) (on_board yes)
-    (property "Reference" "L1" (id 0) (at 110.49 124.46 90)
-      (effects (font (size 1.27 1.27)) (justify left))
-    )
-    (property "Value" "6.8uH" (id 1) (at 113.03 128.27 90)
-      (effects (font (size 1.27 1.27)) (justify left))
-    )
-    (property "Footprint" "iclr:INDM8681X400N" (id 2) (at 110.49 127 0)
-      (effects (font (size 1.27 1.27)) hide)
-    )
-    (property "Datasheet" "~" (id 3) (at 110.49 127 0)
-      (effects (font (size 1.27 1.27)) hide)
-    )
-    (pin "1")
-    (pin "2")
-  )
-  (symbol (lib_id "Device:C_Small") (at 119.38 127 90) (unit 1)
-    (in_bom yes) (on_board yes)
-    (property "Reference" "C6" (id 0) (at 120.65 124.46 90)
-      (effects (font (size 1.27 1.27)) (justify left))
-    )
-    (property "Value" "0.1uF" (id 1) (at 123.19 129.54 90)
-      (effects (font (size 1.27 1.27)) (justify left))
-    )
-    (property "Footprint" "Capacitor_SMD:C_0603_1608Metric" (id 2) (at 119.38 127 0)
-      (effects (font (size 1.27 1.27)) hide)
-    )
-    (property "Datasheet" "~" (id 3) (at 119.38 127 0)
+  (symbol (lib_id "Device:L") (at 97.79 127 90) (unit 1)
+    (in_bom yes) (on_board yes)
+    (property "Reference" "L1" (id 0) (at 97.79 124.46 90)
+      (effects (font (size 1.27 1.27)) (justify left))
+    )
+    (property "Value" "6.8uH" (id 1) (at 100.33 128.27 90)
+      (effects (font (size 1.27 1.27)) (justify left))
+    )
+    (property "Footprint" "iclr:INDM8681X400N" (id 2) (at 97.79 127 0)
+      (effects (font (size 1.27 1.27)) hide)
+    )
+    (property "Datasheet" "~" (id 3) (at 97.79 127 0)
+      (effects (font (size 1.27 1.27)) hide)
+    )
+    (pin "1")
+    (pin "2")
+  )
+  (symbol (lib_id "Device:C_Small") (at 106.68 127 90) (unit 1)
+    (in_bom yes) (on_board yes)
+    (property "Reference" "C6" (id 0) (at 107.95 124.46 90)
+      (effects (font (size 1.27 1.27)) (justify left))
+    )
+    (property "Value" "0.1uF" (id 1) (at 110.49 129.54 90)
+      (effects (font (size 1.27 1.27)) (justify left))
+    )
+    (property "Footprint" "Capacitor_SMD:C_0603_1608Metric" (id 2) (at 106.68 127 0)
+      (effects (font (size 1.27 1.27)) hide)
+    )
+    (property "Datasheet" "~" (id 3) (at 106.68 127 0)
       (effects (font (size 1.27 1.27)) hide)
     )
@@
     (pin "1")
   )
+  (symbol (lib_id "Device:R_Small") (at 90.17 127 90) (unit 1)
+    (in_bom yes) (on_board yes)
+    (property "Reference" "RSR1" (id 0) (at 90.17 122.0216 90))
+    (property "Value" "10m" (id 1) (at 90.17 124.333 90))
+    (property "Footprint" "Resistor_SMD:R_0603_1608Metric" (id 2) (at 90.17 127 0)
+      (effects (font (size 1.27 1.27)) hide)
+    )
+    (property "Datasheet" "~" (id 3) (at 90.17 127 0)
+      (effects (font (size 1.27 1.27)) hide)
+    )
+    (pin "1")
+    (pin "2")
+  )
   (symbol (lib_id "Connector:Conn_01x02_Male") (at 79.4004 184.3024 180) (unit 1)
     (in_bom yes) (on_board yes)
@@
     )
     (pin "1")
-    (pin "2")
-  )
-  (symbol (lib_id "iclr:FCSL110R010FER") (at 87.63 127 0) (unit 1)
-    (in_bom yes) (on_board yes) (fields_autoplaced)
-    (property "Reference" "RSR1" (id 0) (at 96.52 122.081 0))
-    (property "Value" "FCSL110R010FER" (id 1) (at 96.52 124.6179 0))
-    (property "Footprint" "iclr:RESC50110X70N" (id 2) (at 101.6 125.73 0)
-      (effects (font (size 1.27 1.27)) (justify left) hide)
-    )
-    (property "Datasheet" "https://www.ohmite.com/assets/docs/res_fcsl.pdf?r=false" (id 3) (at 101.6 128.27 0)
-      (effects (font (size 1.27 1.27)) (justify left) hide)
-    )
-    (property "Description" "Arcol Ohmite 10m, 4320 Metal Foil SMD Resistor +/-1% 5W - FCSL110R010FER" (id 4) (at 101.6 130.81 0)
-      (effects (font (size 1.27 1.27)) (justify left) hide)
-    )
-    (property "Height" "0.5" (id 5) (at 101.6 133.35 0)
-      (effects (font (size 1.27 1.27)) (justify left) hide)
-    )
-    (property "Manufacturer_Name" "Ohmite" (id 6) (at 101.6 135.89 0)
-      (effects (font (size 1.27 1.27)) (justify left) hide)
-    )
-    (property "Manufacturer_Part_Number" "FCSL110R010FER" (id 7) (at 101.6 138.43 0)
-      (effects (font (size 1.27 1.27)) (justify left) hide)
-    )
-    (property "Mouser Part Number" "588-FCSL110R010FER" (id 8) (at 101.6 140.97 0)
-      (effects (font (size 1.27 1.27)) (justify left) hide)
-    )
-    (property "Mouser Price/Stock" "https://www.mouser.co.uk/ProductDetail/Ohmite/FCSL110R010FER/?qs=MhoRK8A7%252BtW%2F5XGSjsF0ww%3D%3D" (id 9) (at 101.6 143.51 0)
-      (effects (font (size 1.27 1.27)) (justify left) hide)
-    )
-    (property "Arrow Part Number" "" (id 10) (at 101.6 146.05 0)
-      (effects (font (size 1.27 1.27)) (justify left) hide)
-    )
-    (property "Arrow Price/Stock" "" (id 11) (at 101.6 148.59 0)
-      (effects (font (size 1.27 1.27)) (justify left) hide)
-    )
-    (pin "1")

Commit message: swapping mosfets the right way around
Connections:
- net System: now also Q3.3; no longer Q3.2
- net at C3.1, C33.2, IC1.2 (ACP)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: now also Q2.2; no longer Q2.3
- net at J5.1 (Pin_1), J5.2 (Pin_2), PowerLED1.2 (A)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: now also Q1.2; no longer Q1.3
- net Q1-D renamed Q1-S
- net Q1-S: now also Q1.3, Q2.3; no longer Q1.2, Q2.2
- net Q3-S renamed Q3-D
- net Q3-D: now also Q3.2; no longer Q3.3
Other:
- moved on the sheet: Q1, Q2, Q3

Commit message: dan's review
Parts:
- added C21: 0.1uF, Capacitor_SMD:C_0603_1608Metric, symbol Device:C_Small
- C32: value 22uF -> 10uF; footprint Capacitor_SMD:C_1206_3216Metric -> Capacitor_SMD:C_0805_2012Metric
- C8, C9: footprint Capacitor_SMD:C_0805_2012Metric -> Capacitor_SMD:C_0805_2012Metric_Pad1.18x1.45mm_HandSolder
- R10: value 430k -> 10.5k
- R9: value 9.31k -> 2.7k
Connections:
- net GND: now also C12.2, C13.2, C16.2, C8.2, C9.2, C21.2; no longer C12.1, C13.1, C16.1, C8.1, C9.1
- net Q3-D: now also C11.2, C12.1, C13.1, IC1.13 (SRN); no longer C11.1, C12.2, C13.2, IC1.14 (SRP)
- net SRP: now also C11.1, IC1.14 (SRP); no longer C11.2, IC1.13 (SRN)
- net System: now also C8.1, C9.1, C21.1; no longer C8.2, C9.2
- net at R20.1: now also C16.1; no longer C16.2
Other:
- moved on the sheet: C10
