File: Powerboard/Hardware/usb__uart.kicad_sch (KiCad schematic)
At the start: 24 parts, among them IC2 CP2102, J8 USB_C_Receptacle_USB2.0, U11 LTC4411, U4 SC4216H

Commit message: re-layed out pdu to improve buck smps stability
Parts:
- removed TP25: TestPoint, TestPoint:TestPoint_Pad_D1.0mm, symbol Connector:TestPoint
Changed lines of the file:
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@@
   (junction (at 115.57 58.42) (diameter 0) (color 0 0 0 0)
-  )
-  (junction (at 114.3 78.74) (diameter 0) (color 0 0 0 0)
   )
   (junction (at 270.51 121.92) (diameter 0) (color 0 0 0 0)
@@
   (no_connect (at 152.4 116.84))
   (no_connect (at 172.72 93.98))
-  (wire (pts (xy 114.3 78.74) (xy 115.57 78.74))
+  (wire (pts (xy 111.76 78.74) (xy 115.57 78.74))
     (stroke (width 0) (type default) (color 0 0 0 0))
   )
@@
   )
   (wire (pts (xy 124.46 96.52) (xy 124.46 123.19))
-    (stroke (width 0) (type default) (color 0 0 0 0))
-  )
-  (wire (pts (xy 111.76 78.74) (xy 114.3 78.74))
     (stroke (width 0) (type default) (color 0 0 0 0))
   )
@@
     (pin "S1")
   )
-  (symbol (lib_id "Connector:TestPoint") (at 114.3 78.74 0) (unit 1)
-    (in_bom yes) (on_board yes) (fields_autoplaced)
-    (property "Reference" "TP25" (id 0) (at 115.697 74.6033 0)
-      (effects (font (size 1.27 1.27)) (justify left))
-    )
-    (property "Value" "TestPoint" (id 1) (at 115.697 77.1402 0)
-      (effects (font (size 1.27 1.27)) (justify left))
-    )
-    (property "Footprint" "TestPoint:TestPoint_Pad_D1.0mm" (id 2) (at 119.38 78.74 0)
-      (effects (font (size 1.27 1.27)) hide)
-    )
-    (property "Datasheet" "~" (id 3) (at 119.38 78.74 0)
-      (effects (font (size 1.27 1.27)) hide)
-    )
-    (pin "1")
-  )
   (symbol (lib_id "power:GND") (at 80.01 118.7196 0) (unit 1)
