File: Powerboard/Hardware/battchrg.kicad_sch (KiCad schematic)
At the start: 57 parts, among them IC1 BQ24618RGET-iclr, J1 Thermistor Connection 103AT N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, J5 Conn_01x04_Male, J6 Conn_01x02_Male, J7 IsolationSwitch, Q1 RSJ250P10TL, Q2 RSJ250P10TL, Q3 RSJ250P10TL, Q4 RS1G120MN, Q5 RS1G120MN

Commit message: Fixed file location and changed a trace width
Parts:
- added C21: 0.1uF, Capacitor_SMD:C_0603_1608Metric, symbol Device:C_Small
- C32: value 22uF -> 10uF; footprint Capacitor_SMD:C_1206_3216Metric -> Capacitor_SMD:C_0805_2012Metric
- C8, C9: footprint Capacitor_SMD:C_0805_2012Metric -> Capacitor_SMD:C_0805_2012Metric_Pad1.18x1.45mm_HandSolder
- R10: value 430k -> 10.5k
- R9: value 9.31k -> 2.7k
Connections:
- net GND: now also C12.2, C13.2, C16.2, C8.2, C9.2, C21.2; no longer C12.1, C13.1, C16.1, C8.1, C9.1
- net SRP: now also C11.1, IC1.14 (SRP); no longer C11.2, IC1.13 (SRN)
- net System: now also C8.1, C9.1, Q3.3, C21.1; no longer C8.2, C9.2, Q3.2
- net at C3.1, C33.2, IC1.2 (ACP)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: now also Q2.2; no longer Q2.3
- net at R20.1: now also C16.1; no longer C16.2
- net at J5.1 (Pin_1), J5.2 (Pin_2), PowerLED1.2 (A)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: now also Q1.2; no longer Q1.3
- net Q1-D renamed Q1-S
- net Q1-S: now also Q1.3, Q2.3; no longer Q1.2, Q2.2
- net Q3-S renamed Q3-D
- net Q3-D: now also C11.2, C12.1, C13.1, IC1.13 (SRN), Q3.2; no longer C11.1, C12.2, C13.2, IC1.14 (SRP), Q3.3
Other:
- moved on the sheet: C10, Q1, Q2, Q3

Commit message: re-layed out pdu to improve buck smps stability
Parts:
- J1: footprint Connector_JST:JST_XH_B2B-XH-AM_1x02_P2.50mm_Vertical -> Connector_JST:JST_XH_B2B-XH-A_1x02_P2.50mm_Vertical
Changed lines of the file:
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@@
     (property "Reference" "J1" (id 0) (at 170.18 118.11 0))
     (property "Value" "Thermistor Connection 103AT NTC" (id 1) (at 163.83 120.65 0))
-    (property "Footprint" "Connector_JST:JST_XH_B2B-XH-AM_1x02_P2.50mm_Vertical" (id 2) (at 172.72 118.11 0)
+    (property "Footprint" "Connector_JST:JST_XH_B2B-XH-A_1x02_P2.50mm_Vertical" (id 2) (at 172.72 118.11 0)
       (effects (font (size 1.27 1.27)) hide)
     )

Commit message: update
Connections:
- net Q3-D: now also J7.2 (Pin_2); no longer J7.1 (Pin_1)
- net at C31.1, C32.1, J6.2 (Pin_2)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: now also J7.1 (Pin_1); no longer J7.2 (Pin_2)
Other:
- moved on the sheet: J7

Commit message: Changed input filter resistors and changed layout to match
Parts:
- R17: footprint Resistor_SMD:R_0603_1608Metric -> Resistor_SMD:R_1206_3216Metric
- R20: footprint Resistor_SMD:R_0603_1608Metric -> Resistor_SMD:R_2010_5025Metric
Changed lines of the file:
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@@
       (effects (font (size 1.27 1.27)) (justify left))
     )
-    (property "Footprint" "Resistor_SMD:R_0603_1608Metric" (id 2) (at 132.08 107.95 0)
+    (property "Footprint" "Resistor_SMD:R_1206_3216Metric" (id 2) (at 132.08 107.95 0)
       (effects (font (size 1.27 1.27)) hide)
     )
@@
       (effects (font (size 1.27 1.27)) (justify left))
     )
-    (property "Footprint" "Resistor_SMD:R_0603_1608Metric" (id 2) (at 73.66 59.69 0)
+    (property "Footprint" "Resistor_SMD:R_2010_5025Metric" (id 2) (at 73.66 59.69 0)
       (effects (font (size 1.27 1.27)) hide)
     )

Commit message: updated pins and new layout
Parts:
- R28, R29: footprint Resistor_SMD:R_0603_1608Metric -> Resistor_SMD:R_0805_2012Metric
Changed lines of the file:
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@@
       (effects (font (size 1.27 1.27)) (justify left))
     )
-    (property "Footprint" "Resistor_SMD:R_0603_1608Metric" (id 2) (at 67.31 46.99 0)
+    (property "Footprint" "Resistor_SMD:R_0805_2012Metric" (id 2) (at 67.31 46.99 0)
       (effects (font (size 1.27 1.27)) hide)
     )
@@
       (effects (font (size 1.27 1.27)) (justify left))
     )
-    (property "Footprint" "Resistor_SMD:R_0603_1608Metric" (id 2) (at 57.15 137.16 0)
+    (property "Footprint" "Resistor_SMD:R_0805_2012Metric" (id 2) (at 57.15 137.16 0)
       (effects (font (size 1.27 1.27)) hide)
     )
