File: Powerboard/Hardware/powerboard_sc21_as25.kicad_sch (KiCad schematic)
At the start: 45 parts, among them J10 Conn_01x04_Male, J11 Conn_01x03_MountingPin, J2 Conn_01x02_Male, J3 Conn_01x02_Male, J4 Conn_01x08_Male, J9 Conn_Coaxial, Q6 MMDT2222A, Q7 RSJ250P10TL, Q8 RSJ250P10TL, U1 LTC4412xS6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

Commit message: update
Parts:
- added TP1: TestPoint, TestPoint:TestPoint_Pad_D1.5mm, symbol Connector:TestPoint
Connections:
- net LPC_24V: now also TP1.1
Changed lines of the file:
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@@
+    (stroke (width 0) (type default) (color 0 0 0 0))
+  )
+  (wire (pts (xy 237.49 53.34) (xy 247.65 53.34))
     (stroke (width 0) (type default) (color 0 0 0 0))
   )
@@
     (pin "2")
   )
+  (symbol (lib_id "Connector:TestPoint") (at 247.65 53.34 0) (unit 1)
+    (in_bom yes) (on_board yes) (fields_autoplaced)
+    (property "Reference" "TP1" (id 0) (at 250.19 48.7679 0)
+      (effects (font (size 1.27 1.27)) (justify left))
+    )
+    (property "Value" "TestPoint" (id 1) (at 250.19 51.3079 0)
+      (effects (font (size 1.27 1.27)) (justify left))
+    )
+    (property "Footprint" "TestPoint:TestPoint_Pad_D1.5mm" (id 2) (at 252.73 53.34 0)
+      (effects (font (size 1.27 1.27)) hide)
+    )
+    (property "Datasheet" "~" (id 3) (at 252.73 53.34 0)
+      (effects (font (size 1.27 1.27)) hide)
+    )
+    (pin "1")
+  )
   (symbol (lib_id "Diode:SM712_SOT23") (at 255.27 149.86 270) (unit 1)
     (in_bom yes) (on_board yes)
@@
       (reference "RSR1") (unit 1) (value "10m") (footprint "Resistor_SMD:R_0603_1608Metric")
     )
+    (path "/75db9b73-547b-44b5-91e6-0aadeadd89fe"
+      (reference "TP1") (unit 1) (value "TestPoint") (footprint "TestPoint:TestPoint_Pad_D1.5mm")
+    )
     (path "/6475a1e6-8bd5-44d3-bfd0-320d530e7f43"
